Commit message: fix: Corregir nombres de joints en SRDF y rutas de Jinja2 en sim.launch.py
- SRDF mm_arm.srdf.xacro: cambiar joint_1..6 por nombres reales del URDF
  (shoulder_pan_joint, shoulder_lift_joint, elbow_joint, wrist_1/2/3_joint)
- SRDF: actualizar disable_collisions con link_0 -> base_link
- sim.launch.py: arreglar cálculo de config_dir para encontrar templates jinja2
  (antes: 3x dirname incorrecto, ahora: dirname directo del path)

Resultado:
- MoveGroup grupo 'arm' ahora tiene 6 joints válidos
- Templates jinja2 se renderizan correctamente
- RViz y Gazebo inician sin errores de rendering
- Sistema listo para planificación de movimiento

File: ros2_ws/src/mm_arm_description/srdf/mm_arm.srdf.xacro (robot description, xacro)
@@ -10,10 +10,10 @@
   <!-- Grupo para el brazo (6 joints rotacionales) -->
   <group name="arm">
-    <joint name="${prefix}joint_1"/>
-    <joint name="${prefix}joint_2"/>
-    <joint name="${prefix}joint_3"/>
-    <joint name="${prefix}joint_4"/>
-    <joint name="${prefix}joint_5"/>
-    <joint name="${prefix}joint_6"/>
+    <joint name="${prefix}shoulder_pan_joint"/>
+    <joint name="${prefix}shoulder_lift_joint"/>
+    <joint name="${prefix}elbow_joint"/>
+    <joint name="${prefix}wrist_1_joint"/>
+    <joint name="${prefix}wrist_2_joint"/>
+    <joint name="${prefix}wrist_3_joint"/>
   </group>
   <!-- Grupo para el gripper (si existe) -->
@@ -28,5 +28,5 @@
   <!-- ==================== DESHABILITAR COLISIONES ==================== -->
   <!-- Deshabilitar colisiones entre links adyacentes (mismo material, no colisionan) -->
-  <disable_collisions link1="${prefix}link_0" link2="${prefix}link_1" reason="Adjacent"/>
+  <disable_collisions link1="${prefix}base_link" link2="${prefix}link_1" reason="Adjacent"/>
   <disable_collisions link1="${prefix}link_1" link2="${prefix}link_2" reason="Adjacent"/>
   <disable_collisions link1="${prefix}link_2" link2="${prefix}link_3" reason="Adjacent"/>
@@ -35,5 +35,5 @@
   <disable_collisions link1="${prefix}link_5" link2="${prefix}link_6" reason="Adjacent"/>
   <!-- Deshabilitar auto-colisiones (el robot no choca consigo mismo típicamente) -->
-  <disable_collisions link1="${prefix}link_0" link2="${prefix}link_2" reason="Non-adjacent"/>
+  <disable_collisions link1="${prefix}base_link" link2="${prefix}link_2" reason="Non-adjacent"/>
   <disable_collisions link1="${prefix}link_1" link2="${prefix}link_3" reason="Non-adjacent"/>
   <disable_collisions link1="${prefix}link_2" link2="${prefix}link_4" reason="Non-adjacent"/>

Commit message: Estabiliza simulacion headless y MoveIt
Evita segfault de Gazebo en entorno headless usando world sin sensores de render y banderas de xacro. Corrige SRDF y kinematics para que MoveIt cargue el end effector y plugins sin errores.

File: ros2_ws/src/mm_arm_description/srdf/mm_arm.srdf.xacro (robot description, xacro)
@@ -7,4 +7,5 @@
   <xacro:property name="prefix" value="$(arg prefix)"/>
   <xacro:property name="scale" value="$(arg scale)"/>
+  <!-- Test minimo: xacro mm_arm.srdf.xacro prefix:=mm_arm_ -->
   <!-- ==================== GRUPOS DE PLANIFICACIÓN ==================== -->
   <!-- Grupo para el brazo (6 joints rotacionales) -->
@@ -16,5 +17,14 @@
     <joint name="${prefix}wrist_2_joint"/>
     <joint name="${prefix}wrist_3_joint"/>
+    <joint name="${prefix}tool_joint"/>
   </group>
+  <group_state name="home" group="arm">
+    <joint name="${prefix}shoulder_pan_joint" value="0.0"/>
+    <joint name="${prefix}shoulder_lift_joint" value="0.0"/>
+    <joint name="${prefix}elbow_joint" value="0.0"/>
+    <joint name="${prefix}wrist_1_joint" value="0.0"/>
+    <joint name="${prefix}wrist_2_joint" value="0.0"/>
+    <joint name="${prefix}wrist_3_joint" value="0.0"/>
+  </group_state>
   <!-- Grupo para el gripper (si existe) -->
   <group name="gripper">
@@ -42,5 +52,6 @@
   <!-- ==================== END EFFECTOR ==================== -->
   <!-- Define el end effector (herramienta/gripper) -->
-  <end_effector name="ee" parent_link="${prefix}link_6" group="gripper"/>
+  <end_effector name="ee" parent_link="${prefix}tool0" parent_group="arm" group="gripper"/>
+  <virtual_joint name="world_joint" type="fixed" parent_frame="world" child_link="${prefix}root_link"/>
   <!-- ==================== JOINT LIMITS OVERRIDE (OPCIONAL) ==================== -->
   <!-- Se pueden redefinir límites aquí si es necesario -->

File: ros2_ws/src/mm_arm_description/urdf/mm_arm.urdf.xacro (robot description, xacro)
@@ -4,7 +4,9 @@
   <xacro:arg name="scale" default="1.0"/>
   <xacro:arg name="controllers_file" default="$(find-pkg-share mm_bringup)/config/arm_controllers.yaml"/>
+  <xacro:arg name="enable_camera" default="true"/>
   <xacro:property name="prefix" value="$(arg prefix)"/>
   <xacro:property name="scale" value="$(arg scale)"/>
   <xacro:property name="controllers_file" value="$(arg controllers_file)"/>
+  <xacro:property name="enable_camera" value="$(arg enable_camera)"/>
   <!-- Geometría provisional; usar scale para iterar rápidamente. -->
   <xacro:property name="link1_len" value="${0.22 * scale}"/>
@@ -303,24 +305,26 @@
     </plugin>
   </gazebo>
-  <gazebo reference="${prefix}ee_camera_link">
-    <sensor name="ee_camera" type="camera">
-      <topic>/mm_arm/camera</topic>
-      <update_rate>30</update_rate>
-      <always_on>1</always_on>
-      <visualize>true</visualize>
-      <camera>
-        <horizontal_fov>1.047</horizontal_fov>
-        <image>
-          <width>640</width>
-          <height>480</height>
-          <format>R8G8B8</format>
-        </image>
-        <clip>
-          <near>0.05</near>
-          <far>20.0</far>
-        </clip>
-      </camera>
-    </sensor>
-  </gazebo>
+  <xacro:if value="${enable_camera}">
+    <gazebo reference="${prefix}ee_camera_link">
+      <sensor name="ee_camera" type="camera">
+        <topic>/mm_arm/camera</topic>
+        <update_rate>30</update_rate>
+        <always_on>1</always_on>
+        <visualize>true</visualize>
+        <camera>
+          <horizontal_fov>1.047</horizontal_fov>
+          <image>
+            <width>640</width>
+            <height>480</height>
+            <format>R8G8B8</format>
+          </image>
+          <clip>
+            <near>0.05</near>
+            <far>20.0</far>
+          </clip>
+        </camera>
+      </sensor>
+    </gazebo>
+  </xacro:if>
   <gazebo reference="${prefix}ee_imu_link">
     <sensor name="ee_imu" type="imu">

File: ros2_ws/src/mm_base_description/urdf/mm_base.urdf.xacro (robot description, xacro)
@@ -4,7 +4,9 @@
   <xacro:arg name="scale" default="1.0"/>
   <xacro:arg name="controllers_file" default="$(find-pkg-share mm_bringup)/config/base_controllers.yaml"/>
+  <xacro:arg name="enable_render_sensors" default="true"/>
   <xacro:property name="prefix" value="$(arg prefix)"/>
   <xacro:property name="scale" value="$(arg scale)"/>
   <xacro:property name="controllers_file" value="$(arg controllers_file)"/>
+  <xacro:property name="enable_render_sensors" value="$(arg enable_render_sensors)"/>
   <!-- Dimensiones ajustables de la base (usar scale para iterar rápido). -->
   <xacro:property name="base_length" value="${0.45 * scale}"/>
@@ -204,53 +206,55 @@
     </plugin>
   </gazebo>
-  <gazebo reference="${prefix}lidar_link">
-    <sensor name="lidar" type="gpu_lidar">
-      <topic>/mm_base/scan</topic>
-      <update_rate>10</update_rate>
-      <ray>
-        <scan>
-          <horizontal>
-            <samples>640</samples>
-            <resolution>1</resolution>
-            <min_angle>-1.396263</min_angle>
-            <max_angle>1.396263</max_angle>
-          </horizontal>
-          <vertical>
-            <samples>1</samples>
+  <xacro:if value="${enable_render_sensors}">
+    <gazebo reference="${prefix}lidar_link">
+      <sensor name="lidar" type="gpu_lidar">
+        <topic>/mm_base/scan</topic>
+        <update_rate>10</update_rate>
+        <ray>
+          <scan>
+            <horizontal>
+              <samples>640</samples>
+              <resolution>1</resolution>
+              <min_angle>-1.396263</min_angle>
+              <max_angle>1.396263</max_angle>
+            </horizontal>
+            <vertical>
+              <samples>1</samples>
+              <resolution>0.01</resolution>
+              <min_angle>0</min_angle>
+              <max_angle>0</max_angle>
+            </vertical>
+          </scan>
+          <range>
+            <min>0.10</min>
+            <max>10.0</max>
             <resolution>0.01</resolution>
-            <min_angle>0</min_angle>
-            <max_angle>0</max_angle>
-          </vertical>
-        </scan>
-        <range>
-          <min>0.10</min>
-          <max>10.0</max>
-          <resolution>0.01</resolution>
-        </range>
-      </ray>
-      <always_on>1</always_on>
-      <visualize>true</visualize>
-    </sensor>
-  </gazebo>
-  <gazebo reference="${prefix}camera_link">
-    <sensor name="camera" type="camera">
-      <topic>/mm_base/camera</topic>
-      <update_rate>30</update_rate>
-      <always_on>1</always_on>
-      <visualize>true</visualize>
-      <camera>
-        <horizontal_fov>1.047</horizontal_fov>
-        <image>
-          <width>640</width>
-          <height>480</height>
-          <format>R8G8B8</format>
-        </image>
-        <clip>
-          <near>0.05</near>
-          <far>50.0</far>
-        </clip>
-      </camera>
-    </sensor>
-  </gazebo>
+          </range>
+        </ray>
+        <always_on>1</always_on>
+        <visualize>true</visualize>
+      </sensor>
+    </gazebo>
+    <gazebo reference="${prefix}camera_link">
+      <sensor name="camera" type="camera">
+        <topic>/mm_base/camera</topic>
+        <update_rate>30</update_rate>
+        <always_on>1</always_on>
+        <visualize>true</visualize>
+        <camera>
+          <horizontal_fov>1.047</horizontal_fov>
+          <image>
+            <width>640</width>
+            <height>480</height>
+            <format>R8G8B8</format>
+          </image>
+          <clip>
+            <near>0.05</near>
+            <far>50.0</far>
+          </clip>
+        </camera>
+      </sensor>
+    </gazebo>
+  </xacro:if>
   <gazebo reference="${prefix}imu_link">
     <sensor name="imu" type="imu">
@@ -260,23 +264,25 @@
     </sensor>
   </gazebo>
-  <gazebo reference="${prefix}nav_camera_link">
-    <sensor name="nav_camera" type="camera">
-      <topic>/mm_base/nav_camera</topic>
-      <update_rate>15</update_rate>
-      <always_on>1</always_on>
-      <visualize>true</visualize>
-      <camera>
-        <horizontal_fov>${nav_camera_fov}</horizontal_fov>
-        <image>
-          <width>${nav_camera_width}</width>
-          <height>${nav_camera_height}</height>
-          <format>R8G8B8</format>
-        </image>
-        <clip>
-          <near>0.1</near>
-          <far>60.0</far>
-        </clip>
-      </camera>
-    </sensor>
-  </gazebo>
+  <xacro:if value="${enable_render_sensors}">
+    <gazebo reference="${prefix}nav_camera_link">
+      <sensor name="nav_camera" type="camera">
+        <topic>/mm_base/nav_camera</topic>
+        <update_rate>15</update_rate>
+        <always_on>1</always_on>
+        <visualize>true</visualize>
+        <camera>
+          <horizontal_fov>${nav_camera_fov}</horizontal_fov>
+          <image>
+            <width>${nav_camera_width}</width>
+            <height>${nav_camera_height}</height>
+            <format>R8G8B8</format>
+          </image>
+          <clip>
+            <near>0.1</near>
+            <far>60.0</far>
+          </clip>
+        </camera>
+      </sensor>
+    </gazebo>
+  </xacro:if>
 </robot>
