Commit message: feat: Enhance joy teleoperation and simulation configuration
- Updated joy_teleop.py to use QoS settings for publishers and subscriptions.
- Renamed warehouse world to empty_box and adjusted lighting and background.
- Added bridge_params.yaml for ROS to Gazebo topic mapping.
- Introduced mm_arm.srdf for arm configuration and joint states.
- Configured moveit controllers, kinematics, planning, and servo parameters.
- Implemented nav2 parameters for simulation with a blank map.
- Created joint_state_aggregator.py to merge joint states from base and arm.
- Added blank map files for navigation simulation.

File: ros2_ws/src/mm_base_description/urdf/mm_base.urdf.xacro (robot description, xacro)
@@ -21,4 +21,9 @@
   <xacro:property name="camera_x" value="${base_length / 2.0 + 0.02 * scale}"/>
   <xacro:property name="camera_z" value="${base_height / 2.0 + 0.10 * scale}"/>
+  <xacro:property name="nav_camera_x" value="${0.0}"/>
+  <xacro:property name="nav_camera_z" value="${base_height / 2.0 + 0.22 * scale}"/>
+  <xacro:property name="nav_camera_fov" value="${1.047}"/>
+  <xacro:property name="nav_camera_width" value="640"/>
+  <xacro:property name="nav_camera_height" value="480"/>
   <xacro:macro name="simple_inertial" params="mass inertia">
     <inertial>
@@ -142,4 +147,25 @@
     <origin xyz="0 0 ${base_height / 2.0}" rpy="0 0 0"/>
   </joint>
+  <link name="${prefix}nav_camera_link">
+    <xacro:simple_inertial mass="0.2" inertia="0.0005"/>
+    <visual>
+      <geometry>
+        <box size="0.05 0.03 0.03"/>
+      </geometry>
+      <material name="CameraBlack">
+        <color rgba="0.05 0.05 0.05 1.0"/>
+      </material>
+    </visual>
+    <collision>
+      <geometry>
+        <box size="0.05 0.03 0.03"/>
+      </geometry>
+    </collision>
+  </link>
+  <joint name="${prefix}nav_camera_joint" type="fixed">
+    <parent link="${prefix}base_link"/>
+    <child link="${prefix}nav_camera_link"/>
+    <origin xyz="${nav_camera_x} 0 ${nav_camera_z}" rpy="0 0 0"/>
+  </joint>
   <!-- ros2_control para la base mecanum -->
   <ros2_control name="mm_base_system" type="system">
@@ -234,3 +260,23 @@
     </sensor>
   </gazebo>
+  <gazebo reference="${prefix}nav_camera_link">
+    <sensor name="nav_camera" type="camera">
+      <topic>/mm_base/nav_camera</topic>
+      <update_rate>15</update_rate>
+      <always_on>1</always_on>
+      <visualize>true</visualize>
+      <camera>
+        <horizontal_fov>${nav_camera_fov}</horizontal_fov>
+        <image>
+          <width>${nav_camera_width}</width>
+          <height>${nav_camera_height}</height>
+          <format>R8G8B8</format>
+        </image>
+        <clip>
+          <near>0.1</near>
+          <far>60.0</far>
+        </clip>
+      </camera>
+    </sensor>
+  </gazebo>
 </robot>

Commit message: Parametriza sensores de render en base
Agrega flags para habilitar lidar/camaras por separado y permite mantener el launch aunque falle un spawner al aislar sensores.

File: ros2_ws/src/mm_base_description/urdf/mm_base.urdf.xacro (robot description, xacro)
@@ -5,8 +5,14 @@
   <xacro:arg name="controllers_file" default="$(find-pkg-share mm_bringup)/config/base_controllers.yaml"/>
   <xacro:arg name="enable_render_sensors" default="true"/>
+  <xacro:arg name="enable_lidar" default="true"/>
+  <xacro:arg name="enable_base_camera" default="true"/>
+  <xacro:arg name="enable_nav_camera" default="true"/>
   <xacro:property name="prefix" value="$(arg prefix)"/>
   <xacro:property name="scale" value="$(arg scale)"/>
   <xacro:property name="controllers_file" value="$(arg controllers_file)"/>
   <xacro:property name="enable_render_sensors" value="$(arg enable_render_sensors)"/>
+  <xacro:property name="enable_lidar" value="$(arg enable_lidar)"/>
+  <xacro:property name="enable_base_camera" value="$(arg enable_base_camera)"/>
+  <xacro:property name="enable_nav_camera" value="$(arg enable_nav_camera)"/>
   <!-- Dimensiones ajustables de la base (usar scale para iterar rápido). -->
   <xacro:property name="base_length" value="${0.45 * scale}"/>
@@ -206,5 +212,5 @@
     </plugin>
   </gazebo>
-  <xacro:if value="${enable_render_sensors}">
+  <xacro:if value="${enable_render_sensors and enable_lidar}">
     <gazebo reference="${prefix}lidar_link">
       <sensor name="lidar" type="gpu_lidar">
@@ -236,4 +242,6 @@
       </sensor>
     </gazebo>
+  </xacro:if>
+  <xacro:if value="${enable_render_sensors and enable_base_camera}">
     <gazebo reference="${prefix}camera_link">
       <sensor name="camera" type="camera">
@@ -264,5 +272,5 @@
     </sensor>
   </gazebo>
-  <xacro:if value="${enable_render_sensors}">
+  <xacro:if value="${enable_render_sensors and enable_nav_camera}">
     <gazebo reference="${prefix}nav_camera_link">
       <sensor name="nav_camera" type="camera">
