Commit message: Reestructura descripcion y controladores del manipulador
Separamos macros para base/brazo y agregamos descripcion combinada para sim_mm. Ajustamos controladores con prefijo/namespace y pasamos a interfaces de velocidad para que gz_ros2_control exponga todos los joints en Gazebo.

File: clean_v2/ros2_ws/src/mm_arm_description/srdf/mm_arm.srdf.xacro (robot description, xacro)
@@ -3,5 +3,29 @@
   <xacro:arg name="prefix" default="mm1_"/>
   <xacro:property name="prefix" value="$(arg prefix)"/>
-  <!-- Placeholder: SRDF minimo para completar la estructura. -->
-  <virtual_joint name="world_joint" type="fixed" parent_frame="world" child_link="${prefix}root_link"/>
+  <group name="arm">
+    <joint name="${prefix}arm_shoulder_pan_joint"/>
+    <joint name="${prefix}arm_shoulder_lift_joint"/>
+    <joint name="${prefix}arm_elbow_joint"/>
+    <joint name="${prefix}arm_wrist_1_joint"/>
+    <joint name="${prefix}arm_wrist_2_joint"/>
+    <joint name="${prefix}arm_wrist_3_joint"/>
+  </group>
+  <group name="gripper">
+    <joint name="${prefix}gripper_joint"/>
+  </group>
+  <group name="mm_arm_full">
+    <group name="arm"/>
+    <group name="gripper"/>
+  </group>
+  <group_state name="home" group="arm">
+    <joint name="${prefix}arm_shoulder_pan_joint" value="0.0"/>
+    <joint name="${prefix}arm_shoulder_lift_joint" value="0.0"/>
+    <joint name="${prefix}arm_elbow_joint" value="0.0"/>
+    <joint name="${prefix}arm_wrist_1_joint" value="0.0"/>
+    <joint name="${prefix}arm_wrist_2_joint" value="0.0"/>
+    <joint name="${prefix}arm_wrist_3_joint" value="0.0"/>
+  </group_state>
+  <end_effector name="ee" parent_link="${prefix}tool0" parent_group="arm" group="gripper"/>
+  <virtual_joint name="world_joint" type="fixed" parent_frame="world" child_link="${prefix}arm_root_link"/>
+  <!-- Prueba minima: xacro mm_arm.srdf.xacro prefix:=mm1_ -->
 </robot>

File: clean_v2/ros2_ws/src/mm_base_description/urdf/mm_base.urdf.xacro (robot description, xacro)
@@ -1,157 +1,52 @@
 <?xml version="1.0"?>
 <robot name="mm_base" xmlns:xacro="http://www.ros.org/wiki/xacro">
+  <xacro:include filename="$(find mm_base_description)/urdf/mm_base_macro.xacro"/>
   <xacro:arg name="prefix" default="mm1_"/>
   <xacro:arg name="namespace" default="mm1"/>
   <xacro:arg name="scale" default="1.0"/>
-  <xacro:arg name="controllers_file" default="$(find-pkg-share mm_bringup)/config/base_controllers.yaml"/>
+  <xacro:arg name="controllers_file" default=""/>
+  <xacro:arg name="enable_ros2_control" default="true"/>
   <xacro:property name="prefix" value="$(arg prefix)"/>
   <xacro:property name="namespace" value="$(arg namespace)"/>
   <xacro:property name="scale" value="$(arg scale)"/>
   <xacro:property name="controllers_file" value="$(arg controllers_file)"/>
-  <xacro:property name="base_length" value="${0.50 * scale}"/>
-  <xacro:property name="base_width" value="${0.35 * scale}"/>
-  <xacro:property name="base_height" value="${0.10 * scale}"/>
-  <xacro:property name="wheel_radius" value="${0.07 * scale}"/>
-  <xacro:property name="wheel_width" value="${0.04 * scale}"/>
-  <xacro:macro name="simple_inertial" params="mass ixz">
-    <inertial>
-      <origin xyz="0 0 0" rpy="0 0 0"/>
-      <mass value="${mass}"/>
-      <inertia ixx="${ixz}" ixy="0" ixz="0" iyy="${ixz}" iyz="0" izz="${ixz}"/>
-    </inertial>
-  </xacro:macro>
-  <link name="${prefix}base_footprint"/>
-  <link name="${prefix}base_link">
-    <xacro:simple_inertial mass="15.0" ixz="0.25"/>
-    <visual>
-      <origin xyz="0 0 ${base_height / 2.0}" rpy="0 0 0"/>
-      <geometry>
-        <box size="${base_length} ${base_width} ${base_height}"/>
-      </geometry>
-      <material name="BaseBlue">
-        <color rgba="0.1 0.2 0.6 1.0"/>
-      </material>
-    </visual>
-    <collision>
-      <origin xyz="0 0 ${base_height / 2.0}" rpy="0 0 0"/>
-      <geometry>
-        <box size="${base_length} ${base_width} ${base_height}"/>
-      </geometry>
-    </collision>
-  </link>
-  <joint name="${prefix}base_footprint_joint" type="fixed">
-    <parent link="${prefix}base_footprint"/>
-    <child link="${prefix}base_link"/>
-    <origin xyz="0 0 ${wheel_radius}" rpy="0 0 0"/>
-  </joint>
-  <link name="${prefix}front_left_wheel_link">
-    <xacro:simple_inertial mass="1.0" ixz="0.01"/>
-    <visual>
-      <geometry>
-        <cylinder radius="${wheel_radius}" length="${wheel_width}"/>
-      </geometry>
-    </visual>
-    <collision>
-      <geometry>
-        <cylinder radius="${wheel_radius}" length="${wheel_width}"/>
-      </geometry>
-    </collision>
-  </link>
-  <link name="${prefix}front_right_wheel_link">
-    <xacro:simple_inertial mass="1.0" ixz="0.01"/>
-    <visual>
-      <geometry>
-        <cylinder radius="${wheel_radius}" length="${wheel_width}"/>
-      </geometry>
-    </visual>
-    <collision>
-      <geometry>
-        <cylinder radius="${wheel_radius}" length="${wheel_width}"/>
-      </geometry>
-    </collision>
-  </link>
-  <link name="${prefix}rear_left_wheel_link">
-    <xacro:simple_inertial mass="1.0" ixz="0.01"/>
-    <visual>
-      <geometry>
-        <cylinder radius="${wheel_radius}" length="${wheel_width}"/>
-      </geometry>
-    </visual>
-    <collision>
-      <geometry>
-        <cylinder radius="${wheel_radius}" length="${wheel_width}"/>
-      </geometry>
-    </collision>
-  </link>
-  <link name="${prefix}rear_right_wheel_link">
-    <xacro:simple_inertial mass="1.0" ixz="0.01"/>
-    <visual>
-      <geometry>
-        <cylinder radius="${wheel_radius}" length="${wheel_width}"/>
-      </geometry>
-    </visual>
-    <collision>
-      <geometry>
-        <cylinder radius="${wheel_radius}" length="${wheel_width}"/>
-      </geometry>
-    </collision>
-  </link>
-  <joint name="${prefix}front_left_wheel_joint" type="continuous">
-    <parent link="${prefix}base_link"/>
-    <child link="${prefix}front_left_wheel_link"/>
-    <origin xyz="${base_length / 2.0} ${base_width / 2.0} ${wheel_radius}" rpy="0 1.5708 0"/>
-    <axis xyz="0 0 1"/>
-  </joint>
-  <joint name="${prefix}front_right_wheel_joint" type="continuous">
-    <parent link="${prefix}base_link"/>
-    <child link="${prefix}front_right_wheel_link"/>
-    <origin xyz="${base_length / 2.0} -${base_width / 2.0} ${wheel_radius}" rpy="0 1.5708 0"/>
-    <axis xyz="0 0 1"/>
-  </joint>
-  <joint name="${prefix}rear_left_wheel_joint" type="continuous">
-    <parent link="${prefix}base_link"/>
-    <child link="${prefix}rear_left_wheel_link"/>
-    <origin xyz="-${base_length / 2.0} ${base_width / 2.0} ${wheel_radius}" rpy="0 1.5708 0"/>
-    <axis xyz="0 0 1"/>
-  </joint>
-  <joint name="${prefix}rear_right_wheel_joint" type="continuous">
-    <parent link="${prefix}base_link"/>
-    <child link="${prefix}rear_right_wheel_link"/>
-    <origin xyz="-${base_length / 2.0} -${base_width / 2.0} ${wheel_radius}" rpy="0 1.5708 0"/>
-    <axis xyz="0 0 1"/>
-  </joint>
-  <ros2_control name="mm_base_system" type="system">
-    <hardware>
-      <plugin>gz_ros2_control/GazeboSimSystem</plugin>
-    </hardware>
-    <joint name="${prefix}front_left_wheel_joint">
-      <command_interface name="velocity"/>
-      <state_interface name="position"/>
-      <state_interface name="velocity"/>
-    </joint>
-    <joint name="${prefix}front_right_wheel_joint">
-      <command_interface name="velocity"/>
-      <state_interface name="position"/>
-      <state_interface name="velocity"/>
-    </joint>
-    <joint name="${prefix}rear_left_wheel_joint">
-      <command_interface name="velocity"/>
-      <state_interface name="position"/>
-      <state_interface name="velocity"/>
-    </joint>
-    <joint name="${prefix}rear_right_wheel_joint">
-      <command_interface name="velocity"/>
-      <state_interface name="position"/>
-      <state_interface name="velocity"/>
-    </joint>
-  </ros2_control>
-  <gazebo>
-    <plugin filename="libgz_ros2_control-system.so" name="gz_ros2_control::GazeboSimROS2ControlPlugin">
-      <ros>
-        <namespace>$(arg namespace)</namespace>
-      </ros>
-      <parameters>${controllers_file}</parameters>
-      <controller_manager_name>controller_manager</controller_manager_name>
-    </plugin>
-  </gazebo>
+  <xacro:mm_base prefix="${prefix}" scale="${scale}"/>
+  <xacro:if value="$(arg enable_ros2_control)">
+    <xacro:if value="$(eval controllers_file != '')">
+      <ros2_control name="mm_base_system" type="system">
+        <hardware>
+          <plugin>gz_ros2_control/GazeboSimSystem</plugin>
+        </hardware>
+        <joint name="${prefix}front_left_wheel_joint">
+          <command_interface name="velocity"/>
+          <state_interface name="position"/>
+          <state_interface name="velocity"/>
+        </joint>
+        <joint name="${prefix}front_right_wheel_joint">
+          <command_interface name="velocity"/>
+          <state_interface name="position"/>
+          <state_interface name="velocity"/>
+        </joint>
+        <joint name="${prefix}rear_left_wheel_joint">
+          <command_interface name="velocity"/>
+          <state_interface name="position"/>
+          <state_interface name="velocity"/>
+        </joint>
+        <joint name="${prefix}rear_right_wheel_joint">
+          <command_interface name="velocity"/>
+          <state_interface name="position"/>
+          <state_interface name="velocity"/>
+        </joint>
+      </ros2_control>
+      <gazebo>
+        <plugin filename="libgz_ros2_control-system.so" name="gz_ros2_control::GazeboSimROS2ControlPlugin">
+          <ros>
+            <namespace>$(arg namespace)</namespace>
+          </ros>
+          <parameters>${controllers_file}</parameters>
+          <controller_manager_name>controller_manager</controller_manager_name>
+        </plugin>
+      </gazebo>
+    </xacro:if>
+  </xacro:if>
 </robot>

File: clean_v2/ros2_ws/src/mm_robot_description/urdf/mm_robot.urdf.xacro (robot description, xacro)
@@ -1,21 +1,54 @@
 <?xml version="1.0"?>
-<robot name="mm_arm" xmlns:xacro="http://www.ros.org/wiki/xacro">
+<robot name="mm_mobile_manipulator" xmlns:xacro="http://www.ros.org/wiki/xacro">
+  <xacro:include filename="$(find mm_base_description)/urdf/mm_base_macro.xacro"/>
   <xacro:include filename="$(find mm_arm_description)/urdf/mm_arm_macro.xacro"/>
   <xacro:arg name="prefix" default="mm1_"/>
-  <xacro:arg name="namespace" default="mm1/arm"/>
+  <xacro:arg name="namespace" default="mm1"/>
   <xacro:arg name="scale" default="1.0"/>
   <xacro:arg name="controllers_file" default=""/>
   <xacro:arg name="enable_ros2_control" default="true"/>
+  <xacro:arg name="arm_x" default="0.0"/>
+  <xacro:arg name="arm_y" default="0.0"/>
+  <xacro:arg name="arm_z" default="0.30"/>
+  <xacro:arg name="arm_roll" default="0.0"/>
+  <xacro:arg name="arm_pitch" default="0.0"/>
+  <xacro:arg name="arm_yaw" default="0.0"/>
   <xacro:property name="prefix" value="$(arg prefix)"/>
   <xacro:property name="namespace" value="$(arg namespace)"/>
   <xacro:property name="scale" value="$(arg scale)"/>
   <xacro:property name="controllers_file" value="$(arg controllers_file)"/>
+  <xacro:mm_base prefix="${prefix}" scale="${scale}"/>
   <xacro:mm_arm prefix="${prefix}" scale="${scale}"/>
+  <joint name="${prefix}base_to_arm_joint" type="fixed">
+    <parent link="${prefix}base_link"/>
+    <child link="${prefix}arm_root_link"/>
+    <origin xyz="$(arg arm_x) $(arg arm_y) $(arg arm_z)" rpy="$(arg arm_roll) $(arg arm_pitch) $(arg arm_yaw)"/>
+  </joint>
   <xacro:if value="$(arg enable_ros2_control)">
     <xacro:if value="$(eval controllers_file != '')">
-      <ros2_control name="mm_arm_system" type="system">
+      <ros2_control name="mm_mobile_system" type="system">
         <hardware>
           <plugin>gz_ros2_control/GazeboSimSystem</plugin>
         </hardware>
+        <joint name="${prefix}front_left_wheel_joint">
+          <command_interface name="velocity"/>
+          <state_interface name="position"/>
+          <state_interface name="velocity"/>
+        </joint>
+        <joint name="${prefix}front_right_wheel_joint">
+          <command_interface name="velocity"/>
+          <state_interface name="position"/>
+          <state_interface name="velocity"/>
+        </joint>
+        <joint name="${prefix}rear_left_wheel_joint">
+          <command_interface name="velocity"/>
+          <state_interface name="position"/>
+          <state_interface name="velocity"/>
+        </joint>
+        <joint name="${prefix}rear_right_wheel_joint">
+          <command_interface name="velocity"/>
+          <state_interface name="position"/>
+          <state_interface name="velocity"/>
+        </joint>
         <joint name="${prefix}arm_shoulder_pan_joint">
           <command_interface name="velocity"/>
