Commit message: fix: alinear ruedas y base del brazo
Ubica los centros de rueda a nivel de base_link y baja el brazo para que quede anclado al chasis.

File: clean_v2/ros2_ws/src/mm_base_description/urdf/mm_base_macro.xacro (robot description, xacro)
@@ -93,5 +93,5 @@
       <parent link="${prefix}base_link"/>
       <child link="${prefix}front_left_wheel_link"/>
-      <origin xyz="${base_length / 2.0} ${base_width / 2.0} ${wheel_radius}" rpy="0 1.5708 0"/>
+      <origin xyz="${base_length / 2.0} ${base_width / 2.0} 0.0" rpy="0 1.5708 0"/>
       <axis xyz="0 0 1"/>
     </joint>
@@ -99,5 +99,5 @@
       <parent link="${prefix}base_link"/>
       <child link="${prefix}front_right_wheel_link"/>
-      <origin xyz="${base_length / 2.0} -${base_width / 2.0} ${wheel_radius}" rpy="0 1.5708 0"/>
+      <origin xyz="${base_length / 2.0} -${base_width / 2.0} 0.0" rpy="0 1.5708 0"/>
       <axis xyz="0 0 1"/>
     </joint>
@@ -105,5 +105,5 @@
       <parent link="${prefix}base_link"/>
       <child link="${prefix}rear_left_wheel_link"/>
-      <origin xyz="-${base_length / 2.0} ${base_width / 2.0} ${wheel_radius}" rpy="0 1.5708 0"/>
+      <origin xyz="-${base_length / 2.0} ${base_width / 2.0} 0.0" rpy="0 1.5708 0"/>
       <axis xyz="0 0 1"/>
     </joint>
@@ -111,5 +111,5 @@
       <parent link="${prefix}base_link"/>
       <child link="${prefix}rear_right_wheel_link"/>
-      <origin xyz="-${base_length / 2.0} -${base_width / 2.0} ${wheel_radius}" rpy="0 1.5708 0"/>
+      <origin xyz="-${base_length / 2.0} -${base_width / 2.0} 0.0" rpy="0 1.5708 0"/>
       <axis xyz="0 0 1"/>
     </joint>

File: clean_v2/ros2_ws/src/mm_robot_description/urdf/mm_robot.urdf.xacro (robot description, xacro)
@@ -10,5 +10,5 @@
   <xacro:arg name="arm_x" default="0.0"/>
   <xacro:arg name="arm_y" default="0.0"/>
-  <xacro:arg name="arm_z" default="0.30"/>
+  <xacro:arg name="arm_z" default="0.05"/>
   <xacro:arg name="arm_roll" default="0.0"/>
   <xacro:arg name="arm_pitch" default="0.0"/>

Commit message: Actualizar metadata y ajustes base/arm
Reemplaza placeholders de maintainer y corrige medidas de base/brazo.

File: clean_v2/ros2_ws/src/mm_base_description/urdf/mm_base_macro.xacro (robot description, xacro)
@@ -13,5 +13,5 @@
     <xacro:property name="wheel_width" value="${0.04 * scale}"/>
     <xacro:property name="base_length" value="${0.50 * scale}"/>
-    <xacro:property name="base_width" value="${0.35 * scale}"/>
+    <xacro:property name="base_width" value="${0.60 * scale}"/>
     <xacro:property name="base_height" value="${0.10 * scale}"/>
     <xacro:property name="base_visual_margin_xy" value="${0.02 * scale}"/>
@@ -24,8 +24,8 @@
     <xacro:property name="base_mount_z" value="${wheel_radius}"/>
     <xacro:property name="wheel_center_z" value="0.0"/>
-    <xacro:property name="wheel_front_x" value="${base_length / 2.0}"/>
-    <xacro:property name="wheel_rear_x" value="${-base_length / 2.0}"/>
-    <xacro:property name="wheel_left_y" value="${base_width / 2.0}"/>
-    <xacro:property name="wheel_right_y" value="${-base_width / 2.0}"/>
+    <xacro:property name="wheel_front_x" value="${base_length / 1.9}"/>
+    <xacro:property name="wheel_rear_x" value="${-base_length / 1.9}"/>
+    <xacro:property name="wheel_left_y" value="${(base_width / 3.5) + wheel_radius}"/>
+    <xacro:property name="wheel_right_y" value="${-(base_width / 3.5) - wheel_radius}"/>
     <link name="${prefix}base_footprint"/>
     <xacro:property name="base_visual_enabled" value="${visual_mode == 'full' or visual_mode == 'base_only'}"/>

File: clean_v2/ros2_ws/src/mm_robot_description/urdf/mm_robot.urdf.xacro (robot description, xacro)
@@ -63,5 +63,5 @@
   <xacro:property name="base_height" value="${0.10 * scale}"/>
   <xacro:property name="arm_mount_height" value="$(arg arm_z)"/>
-  <xacro:property name="arm_mount_z" value="${base_height + arm_mount_height}"/>
+  <xacro:property name="arm_mount_z" value="${(base_height / 2.0) + arm_mount_height}"/>
   <xacro:property name="base_visual_enabled" value="${visual_mode == 'full' or visual_mode == 'base_only'}"/>
   <xacro:property name="lidar_topic" value="$(eval '/' + namespace + '/scan' if namespace != '' else '/scan')"/>
