Commit message: feat(moveit): render SRDF/URDF with consistent namespace and prefix

File: clean_v2/ros2_ws/src/mm_moveit_config/config/mm_robot.srdf.xacro (robot description, xacro)
@@ -2,7 +2,8 @@
 <!-- Autor: Camilo Soto Villegas | Contacto: camilo.soto.v@usach.cl | Proyecto: clean_v2 -->
 <!-- SRDF para configuración MoveIt 2 del manipulador móvil mm -->
-<robot name="mm_robot" xmlns:xacro="http://www.ros.org/wiki/xacro">
+<robot name="mm_mobile_manipulator" xmlns:xacro="http://www.ros.org/wiki/xacro">
   <xacro:arg name="prefix" default="mm1_"/>
   <xacro:arg name="enable_lidar" default="true"/>
+  <xacro:property name="prefix" value="$(arg prefix)"/>
   <!-- ============================================================================= -->
   <!-- GRUPOS DE PLANIFICACIÓN (Planning Groups) -->
@@ -106,4 +107,4 @@
   <!-- ============================================================================= -->
   <!-- Virtual joint: conecta el mundo con la base -->
-  <virtual_joint name="fixed_base" type="fixed" parent_frame="world" child_frame="${prefix}base_footprint" />
+  <virtual_joint name="fixed_base" type="fixed" parent_frame="world" child_link="${prefix}base_footprint" />
 </robot>

Commit message: fix(moveit): align SRDF with URDF links and simplify planning groups

File: clean_v2/ros2_ws/src/mm_moveit_config/config/mm_robot.srdf.xacro (robot description, xacro)
@@ -27,20 +27,8 @@
     <group name="gripper" />
   </group>
-  <!-- Grupo: Base móvil omni -->
-  <group name="base">
-    <joint name="${prefix}front_left_wheel_joint" />
-    <joint name="${prefix}front_right_wheel_joint" />
-    <joint name="${prefix}rear_left_wheel_joint" />
-    <joint name="${prefix}rear_right_wheel_joint" />
-  </group>
-  <!-- Grupo: Sistema completo -->
-  <group name="mm_full_system">
-    <group name="base" />
-    <group name="manipulator" />
-  </group>
   <!-- ============================================================================= -->
   <!-- EFECTOR FINAL (End Effector) -->
   <!-- ============================================================================= -->
-  <end_effector name="gripper_eef" parent_link="${prefix}gripper_link" group="gripper" />
+  <end_effector name="gripper_eef" parent_link="${prefix}tool0" parent_group="arm" group="gripper" />
   <!-- ============================================================================= -->
   <!-- DESABILITAR COLISIONES (Disable Collisions) -->
@@ -69,8 +57,4 @@
   <disable_collisions link1="${prefix}arm_link_5" link2="${prefix}arm_link_6" reason="Adjacent" />
   <disable_collisions link1="${prefix}arm_link_6" link2="${prefix}gripper_link" reason="Adjacent" />
-  <!-- Gripper interno: dedos -->
-  <disable_collisions link1="${prefix}gripper_link" link2="${prefix}gripper_finger_left_link" reason="Adjacent" />
-  <disable_collisions link1="${prefix}gripper_link" link2="${prefix}gripper_finger_right_link" reason="Adjacent" />
-  <disable_collisions link1="${prefix}gripper_finger_left_link" link2="${prefix}gripper_finger_right_link" reason="Never" />
   <!-- Sensores: no incluir en colisiones -->
   <xacro:if value="$(arg enable_lidar)">
