Commit message: feat: integrar camaras y mounts en el robot
Añade camaras base y EE con offsets parametrizables, bridge a ROS y documentacion de sensores.

File: clean_v2/ros2_ws/src/mm_arm_description/urdf/mm_arm.urdf.xacro (robot description, xacro)
@@ -7,9 +7,36 @@
   <xacro:arg name="controllers_file" default=""/>
   <xacro:arg name="enable_ros2_control" default="true"/>
+  <xacro:arg name="ee_cam_mount_x" default="0.02"/>
+  <xacro:arg name="ee_cam_mount_y" default="0.0"/>
+  <xacro:arg name="ee_cam_mount_z" default="0.02"/>
+  <xacro:arg name="ee_cam_mount_roll" default="0.0"/>
+  <xacro:arg name="ee_cam_mount_pitch" default="0.0"/>
+  <xacro:arg name="ee_cam_mount_yaw" default="0.0"/>
+  <xacro:arg name="ee_cam_x" default="0.08"/>
+  <xacro:arg name="ee_cam_y" default="0.0"/>
+  <xacro:arg name="ee_cam_z" default="0.02"/>
+  <xacro:arg name="ee_cam_roll" default="0.0"/>
+  <xacro:arg name="ee_cam_pitch" default="0.0"/>
+  <xacro:arg name="ee_cam_yaw" default="0.0"/>
   <xacro:property name="prefix" value="$(arg prefix)"/>
   <xacro:property name="namespace" value="$(arg namespace)"/>
   <xacro:property name="scale" value="$(arg scale)"/>
   <xacro:property name="controllers_file" value="$(arg controllers_file)"/>
-  <xacro:mm_arm prefix="${prefix}" scale="${scale}"/>
+  <xacro:mm_arm
+    prefix="${prefix}"
+    scale="${scale}"
+    ee_cam_mount_x="$(arg ee_cam_mount_x)"
+    ee_cam_mount_y="$(arg ee_cam_mount_y)"
+    ee_cam_mount_z="$(arg ee_cam_mount_z)"
+    ee_cam_mount_roll="$(arg ee_cam_mount_roll)"
+    ee_cam_mount_pitch="$(arg ee_cam_mount_pitch)"
+    ee_cam_mount_yaw="$(arg ee_cam_mount_yaw)"
+    ee_cam_x="$(arg ee_cam_x)"
+    ee_cam_y="$(arg ee_cam_y)"
+    ee_cam_z="$(arg ee_cam_z)"
+    ee_cam_roll="$(arg ee_cam_roll)"
+    ee_cam_pitch="$(arg ee_cam_pitch)"
+    ee_cam_yaw="$(arg ee_cam_yaw)"
+  />
   <xacro:if value="$(arg enable_ros2_control)">
     <xacro:if value="$(eval controllers_file != '')">

File: clean_v2/ros2_ws/src/mm_arm_description/urdf/mm_arm_macro.xacro (robot description, xacro)
@@ -8,5 +8,5 @@
     </inertial>
   </xacro:macro>
-  <xacro:macro name="mm_arm" params="prefix scale">
+  <xacro:macro name="mm_arm" params="prefix scale ee_cam_mount_x ee_cam_mount_y ee_cam_mount_z ee_cam_mount_roll ee_cam_mount_pitch ee_cam_mount_yaw ee_cam_x ee_cam_y ee_cam_z ee_cam_roll ee_cam_pitch ee_cam_yaw">
     <xacro:property name="link1_len" value="${0.22 * scale}"/>
     <xacro:property name="link2_len" value="${0.22 * scale}"/>
@@ -174,4 +174,40 @@
       <origin xyz="0 0 ${link6_len}" rpy="0 0 0"/>
     </joint>
+    <link name="${prefix}ee_cam_mount_link">
+      <xacro:mm_arm_simple_inertial mass="0.2" inertia="0.001" origin_z="0.0"/>
+      <visual>
+        <geometry>
+          <cylinder radius="0.015" length="0.03"/>
+        </geometry>
+      </visual>
+      <collision>
+        <geometry>
+          <cylinder radius="0.015" length="0.03"/>
+        </geometry>
+      </collision>
+    </link>
+    <joint name="${prefix}ee_cam_mount_joint" type="fixed">
+      <parent link="${prefix}tool0"/>
+      <child link="${prefix}ee_cam_mount_link"/>
+      <origin xyz="${ee_cam_mount_x} ${ee_cam_mount_y} ${ee_cam_mount_z}" rpy="${ee_cam_mount_roll} ${ee_cam_mount_pitch} ${ee_cam_mount_yaw}"/>
+    </joint>
+    <link name="${prefix}ee_cam_link">
+      <xacro:mm_arm_simple_inertial mass="0.2" inertia="0.001" origin_z="0.0"/>
+      <visual>
+        <geometry>
+          <box size="0.04 0.03 0.03"/>
+        </geometry>
+      </visual>
+      <collision>
+        <geometry>
+          <box size="0.04 0.03 0.03"/>
+        </geometry>
+      </collision>
+    </link>
+    <joint name="${prefix}ee_cam_joint" type="fixed">
+      <parent link="${prefix}ee_cam_mount_link"/>
+      <child link="${prefix}ee_cam_link"/>
+      <origin xyz="${ee_cam_x} ${ee_cam_y} ${ee_cam_z}" rpy="${ee_cam_roll} ${ee_cam_pitch} ${ee_cam_yaw}"/>
+    </joint>
     <link name="${prefix}gripper_link">
       <xacro:mm_arm_simple_inertial mass="0.2" inertia="0.0005" origin_z="0.0"/>

File: clean_v2/ros2_ws/src/mm_base_description/urdf/mm_base.urdf.xacro (robot description, xacro)
@@ -7,9 +7,60 @@
   <xacro:arg name="controllers_file" default=""/>
   <xacro:arg name="enable_ros2_control" default="true"/>
+  <xacro:arg name="cam_front_x" default="0.26"/>
+  <xacro:arg name="cam_front_y" default="0.0"/>
+  <xacro:arg name="cam_front_z" default="0.12"/>
+  <xacro:arg name="cam_front_roll" default="0.0"/>
+  <xacro:arg name="cam_front_pitch" default="0.0"/>
+  <xacro:arg name="cam_front_yaw" default="0.0"/>
+  <xacro:arg name="cam_left_x" default="0.0"/>
+  <xacro:arg name="cam_left_y" default="0.185"/>
+  <xacro:arg name="cam_left_z" default="0.12"/>
+  <xacro:arg name="cam_left_roll" default="0.0"/>
+  <xacro:arg name="cam_left_pitch" default="0.0"/>
+  <xacro:arg name="cam_left_yaw" default="1.5708"/>
+  <xacro:arg name="cam_right_x" default="0.0"/>
+  <xacro:arg name="cam_right_y" default="-0.185"/>
+  <xacro:arg name="cam_right_z" default="0.12"/>
+  <xacro:arg name="cam_right_roll" default="0.0"/>
+  <xacro:arg name="cam_right_pitch" default="0.0"/>
+  <xacro:arg name="cam_right_yaw" default="-1.5708"/>
+  <xacro:arg name="cam_rear_x" default="-0.26"/>
+  <xacro:arg name="cam_rear_y" default="0.0"/>
+  <xacro:arg name="cam_rear_z" default="0.12"/>
+  <xacro:arg name="cam_rear_roll" default="0.0"/>
+  <xacro:arg name="cam_rear_pitch" default="0.0"/>
+  <xacro:arg name="cam_rear_yaw" default="3.1416"/>
   <xacro:property name="prefix" value="$(arg prefix)"/>
   <xacro:property name="namespace" value="$(arg namespace)"/>
   <xacro:property name="scale" value="$(arg scale)"/>
   <xacro:property name="controllers_file" value="$(arg controllers_file)"/>
-  <xacro:mm_base prefix="${prefix}" scale="${scale}"/>
+  <xacro:mm_base
+    prefix="${prefix}"
+    scale="${scale}"
+    cam_front_x="$(arg cam_front_x)"
+    cam_front_y="$(arg cam_front_y)"
+    cam_front_z="$(arg cam_front_z)"
+    cam_front_roll="$(arg cam_front_roll)"
+    cam_front_pitch="$(arg cam_front_pitch)"
+    cam_front_yaw="$(arg cam_front_yaw)"
+    cam_left_x="$(arg cam_left_x)"
+    cam_left_y="$(arg cam_left_y)"
+    cam_left_z="$(arg cam_left_z)"
+    cam_left_roll="$(arg cam_left_roll)"
+    cam_left_pitch="$(arg cam_left_pitch)"
+    cam_left_yaw="$(arg cam_left_yaw)"
+    cam_right_x="$(arg cam_right_x)"
+    cam_right_y="$(arg cam_right_y)"
+    cam_right_z="$(arg cam_right_z)"
+    cam_right_roll="$(arg cam_right_roll)"
+    cam_right_pitch="$(arg cam_right_pitch)"
+    cam_right_yaw="$(arg cam_right_yaw)"
+    cam_rear_x="$(arg cam_rear_x)"
+    cam_rear_y="$(arg cam_rear_y)"
+    cam_rear_z="$(arg cam_rear_z)"
+    cam_rear_roll="$(arg cam_rear_roll)"
+    cam_rear_pitch="$(arg cam_rear_pitch)"
+    cam_rear_yaw="$(arg cam_rear_yaw)"
+  />
   <xacro:if value="$(arg enable_ros2_control)">
     <xacro:if value="$(eval controllers_file != '')">

File: clean_v2/ros2_ws/src/mm_base_description/urdf/mm_base_macro.xacro (robot description, xacro)
@@ -8,5 +8,5 @@
     </inertial>
   </xacro:macro>
-  <xacro:macro name="mm_base" params="prefix scale">
+  <xacro:macro name="mm_base" params="prefix scale cam_front_x cam_front_y cam_front_z cam_front_roll cam_front_pitch cam_front_yaw cam_left_x cam_left_y cam_left_z cam_left_roll cam_left_pitch cam_left_yaw cam_right_x cam_right_y cam_right_z cam_right_roll cam_right_pitch cam_right_yaw cam_rear_x cam_rear_y cam_rear_z cam_rear_roll cam_rear_pitch cam_rear_yaw">
     <xacro:property name="base_length" value="${0.50 * scale}"/>
     <xacro:property name="base_width" value="${0.35 * scale}"/>
@@ -114,4 +114,76 @@
       <axis xyz="0 0 1"/>
     </joint>
+    <link name="${prefix}cam_front_link">
+      <xacro:mm_base_simple_inertial mass="0.2" ixz="0.001"/>
+      <visual>
+        <geometry>
+          <box size="0.04 0.03 0.03"/>
+        </geometry>
+      </visual>
+      <collision>
+        <geometry>
+          <box size="0.04 0.03 0.03"/>
+        </geometry>
+      </collision>
+    </link>
+    <joint name="${prefix}cam_front_joint" type="fixed">
+      <parent link="${prefix}base_link"/>
+      <child link="${prefix}cam_front_link"/>
+      <origin xyz="${cam_front_x} ${cam_front_y} ${cam_front_z}" rpy="${cam_front_roll} ${cam_front_pitch} ${cam_front_yaw}"/>
+    </joint>
+    <link name="${prefix}cam_left_link">
+      <xacro:mm_base_simple_inertial mass="0.2" ixz="0.001"/>
+      <visual>
+        <geometry>
+          <box size="0.04 0.03 0.03"/>
+        </geometry>
+      </visual>
+      <collision>
+        <geometry>
+          <box size="0.04 0.03 0.03"/>
+        </geometry>
+      </collision>
+    </link>
+    <joint name="${prefix}cam_left_joint" type="fixed">
+      <parent link="${prefix}base_link"/>
+      <child link="${prefix}cam_left_link"/>
+      <origin xyz="${cam_left_x} ${cam_left_y} ${cam_left_z}" rpy="${cam_left_roll} ${cam_left_pitch} ${cam_left_yaw}"/>
+    </joint>
+    <link name="${prefix}cam_right_link">
+      <xacro:mm_base_simple_inertial mass="0.2" ixz="0.001"/>
+      <visual>
+        <geometry>
+          <box size="0.04 0.03 0.03"/>
+        </geometry>
+      </visual>
+      <collision>
+        <geometry>
+          <box size="0.04 0.03 0.03"/>
+        </geometry>
+      </collision>
+    </link>
+    <joint name="${prefix}cam_right_joint" type="fixed">
+      <parent link="${prefix}base_link"/>
+      <child link="${prefix}cam_right_link"/>
+      <origin xyz="${cam_right_x} ${cam_right_y} ${cam_right_z}" rpy="${cam_right_roll} ${cam_right_pitch} ${cam_right_yaw}"/>
+    </joint>
+    <link name="${prefix}cam_rear_link">
+      <xacro:mm_base_simple_inertial mass="0.2" ixz="0.001"/>
+      <visual>
+        <geometry>
+          <box size="0.04 0.03 0.03"/>
+        </geometry>
+      </visual>
+      <collision>
+        <geometry>
+          <box size="0.04 0.03 0.03"/>
+        </geometry>
+      </collision>
+    </link>
+    <joint name="${prefix}cam_rear_joint" type="fixed">
+      <parent link="${prefix}base_link"/>
+      <child link="${prefix}cam_rear_link"/>
+      <origin xyz="${cam_rear_x} ${cam_rear_y} ${cam_rear_z}" rpy="${cam_rear_roll} ${cam_rear_pitch} ${cam_rear_yaw}"/>
+    </joint>
   </xacro:macro>
 </robot>

File: clean_v2/ros2_ws/src/mm_robot_description/urdf/mm_robot.urdf.xacro (robot description, xacro)
@@ -18,4 +18,40 @@
   <xacro:arg name="lidar_y" default="0.0"/>
   <xacro:arg name="lidar_z" default="0.15"/>
+  <xacro:arg name="cam_front_x" default="0.26"/>
+  <xacro:arg name="cam_front_y" default="0.0"/>
+  <xacro:arg name="cam_front_z" default="0.12"/>
+  <xacro:arg name="cam_front_roll" default="0.0"/>
+  <xacro:arg name="cam_front_pitch" default="0.0"/>
+  <xacro:arg name="cam_front_yaw" default="0.0"/>
+  <xacro:arg name="cam_left_x" default="0.0"/>
+  <xacro:arg name="cam_left_y" default="0.185"/>
+  <xacro:arg name="cam_left_z" default="0.12"/>
+  <xacro:arg name="cam_left_roll" default="0.0"/>
+  <xacro:arg name="cam_left_pitch" default="0.0"/>
+  <xacro:arg name="cam_left_yaw" default="1.5708"/>
+  <xacro:arg name="cam_right_x" default="0.0"/>
+  <xacro:arg name="cam_right_y" default="-0.185"/>
+  <xacro:arg name="cam_right_z" default="0.12"/>
+  <xacro:arg name="cam_right_roll" default="0.0"/>
+  <xacro:arg name="cam_right_pitch" default="0.0"/>
+  <xacro:arg name="cam_right_yaw" default="-1.5708"/>
+  <xacro:arg name="cam_rear_x" default="-0.26"/>
+  <xacro:arg name="cam_rear_y" default="0.0"/>
+  <xacro:arg name="cam_rear_z" default="0.12"/>
+  <xacro:arg name="cam_rear_roll" default="0.0"/>
+  <xacro:arg name="cam_rear_pitch" default="0.0"/>
+  <xacro:arg name="cam_rear_yaw" default="3.1416"/>
+  <xacro:arg name="ee_cam_mount_x" default="0.02"/>
+  <xacro:arg name="ee_cam_mount_y" default="0.0"/>
+  <xacro:arg name="ee_cam_mount_z" default="0.02"/>
+  <xacro:arg name="ee_cam_mount_roll" default="0.0"/>
+  <xacro:arg name="ee_cam_mount_pitch" default="0.0"/>
+  <xacro:arg name="ee_cam_mount_yaw" default="0.0"/>
+  <xacro:arg name="ee_cam_x" default="0.08"/>
+  <xacro:arg name="ee_cam_y" default="0.0"/>
+  <xacro:arg name="ee_cam_z" default="0.02"/>
+  <xacro:arg name="ee_cam_roll" default="0.0"/>
+  <xacro:arg name="ee_cam_pitch" default="0.0"/>
+  <xacro:arg name="ee_cam_yaw" default="0.0"/>
   <xacro:property name="prefix" value="$(arg prefix)"/>
   <xacro:property name="namespace" value="$(arg namespace)"/>
@@ -23,6 +59,54 @@
   <xacro:property name="controllers_file" value="$(arg controllers_file)"/>
   <xacro:property name="lidar_topic" value="$(eval '/' + namespace + '/scan' if namespace != '' else '/scan')"/>
-  <xacro:mm_base prefix="${prefix}" scale="${scale}"/>
-  <xacro:mm_arm prefix="${prefix}" scale="${scale}"/>
+  <xacro:property name="camera_topic_prefix" value="$(eval '/' + namespace + '/camera' if namespace != '' else '/camera')"/>
+  <xacro:property name="cam_front_topic" value="$(eval camera_topic_prefix + '/front/image')"/>
+  <xacro:property name="cam_left_topic" value="$(eval camera_topic_prefix + '/left/image')"/>
+  <xacro:property name="cam_right_topic" value="$(eval camera_topic_prefix + '/right/image')"/>
+  <xacro:property name="cam_rear_topic" value="$(eval camera_topic_prefix + '/rear/image')"/>
+  <xacro:property name="ee_cam_topic" value="$(eval camera_topic_prefix + '/ee/image')"/>
+  <xacro:mm_base
+    prefix="${prefix}"
+    scale="${scale}"
+    cam_front_x="$(arg cam_front_x)"
+    cam_front_y="$(arg cam_front_y)"
+    cam_front_z="$(arg cam_front_z)"
+    cam_front_roll="$(arg cam_front_roll)"
+    cam_front_pitch="$(arg cam_front_pitch)"
+    cam_front_yaw="$(arg cam_front_yaw)"
+    cam_left_x="$(arg cam_left_x)"
+    cam_left_y="$(arg cam_left_y)"
+    cam_left_z="$(arg cam_left_z)"
+    cam_left_roll="$(arg cam_left_roll)"
+    cam_left_pitch="$(arg cam_left_pitch)"
+    cam_left_yaw="$(arg cam_left_yaw)"
+    cam_right_x="$(arg cam_right_x)"
+    cam_right_y="$(arg cam_right_y)"
+    cam_right_z="$(arg cam_right_z)"
+    cam_right_roll="$(arg cam_right_roll)"
+    cam_right_pitch="$(arg cam_right_pitch)"
+    cam_right_yaw="$(arg cam_right_yaw)"
+    cam_rear_x="$(arg cam_rear_x)"
+    cam_rear_y="$(arg cam_rear_y)"
+    cam_rear_z="$(arg cam_rear_z)"
+    cam_rear_roll="$(arg cam_rear_roll)"
+    cam_rear_pitch="$(arg cam_rear_pitch)"
+    cam_rear_yaw="$(arg cam_rear_yaw)"
+  />
+  <xacro:mm_arm
+    prefix="${prefix}"
+    scale="${scale}"
+    ee_cam_mount_x="$(arg ee_cam_mount_x)"
+    ee_cam_mount_y="$(arg ee_cam_mount_y)"
+    ee_cam_mount_z="$(arg ee_cam_mount_z)"
+    ee_cam_mount_roll="$(arg ee_cam_mount_roll)"
+    ee_cam_mount_pitch="$(arg ee_cam_mount_pitch)"
+    ee_cam_mount_yaw="$(arg ee_cam_mount_yaw)"
+    ee_cam_x="$(arg ee_cam_x)"
+    ee_cam_y="$(arg ee_cam_y)"
+    ee_cam_z="$(arg ee_cam_z)"
+    ee_cam_roll="$(arg ee_cam_roll)"
+    ee_cam_pitch="$(arg ee_cam_pitch)"
+    ee_cam_yaw="$(arg ee_cam_yaw)"
+  />
   <joint name="${prefix}base_to_arm_joint" type="fixed">
     <parent link="${prefix}base_link"/>
@@ -82,4 +166,99 @@
     </gazebo>
   </xacro:if>
+  <gazebo reference="${prefix}cam_front_link">
+    <sensor name="${prefix}cam_front" type="camera">
+      <pose>0 0 0 0 0 0</pose>
+      <update_rate>15</update_rate>
+      <topic>${cam_front_topic}</topic>
+      <camera>
+        <horizontal_fov>1.3962634</horizontal_fov>
+        <image>
+          <width>640</width>
+          <height>480</height>
+          <format>R8G8B8</format>
+        </image>
+        <clip>
+          <near>0.05</near>
+          <far>20.0</far>
+        </clip>
+      </camera>
+    </sensor>
+  </gazebo>
+  <gazebo reference="${prefix}cam_left_link">
+    <sensor name="${prefix}cam_left" type="camera">
+      <pose>0 0 0 0 0 0</pose>
+      <update_rate>15</update_rate>
+      <topic>${cam_left_topic}</topic>
+      <camera>
+        <horizontal_fov>1.3962634</horizontal_fov>
+        <image>
+          <width>640</width>
+          <height>480</height>
+          <format>R8G8B8</format>
+        </image>
+        <clip>
+          <near>0.05</near>
+          <far>20.0</far>
+        </clip>
+      </camera>
+    </sensor>
+  </gazebo>
+  <gazebo reference="${prefix}cam_right_link">
+    <sensor name="${prefix}cam_right" type="camera">
+      <pose>0 0 0 0 0 0</pose>
+      <update_rate>15</update_rate>
+      <topic>${cam_right_topic}</topic>
+      <camera>
+        <horizontal_fov>1.3962634</horizontal_fov>
+        <image>
+          <width>640</width>
+          <height>480</height>
+          <format>R8G8B8</format>
+        </image>
+        <clip>
+          <near>0.05</near>
+          <far>20.0</far>
+        </clip>
+      </camera>
+    </sensor>
+  </gazebo>
+  <gazebo reference="${prefix}cam_rear_link">
+    <sensor name="${prefix}cam_rear" type="camera">
+      <pose>0 0 0 0 0 0</pose>
+      <update_rate>15</update_rate>
+      <topic>${cam_rear_topic}</topic>
+      <camera>
+        <horizontal_fov>1.3962634</horizontal_fov>
+        <image>
+          <width>640</width>
+          <height>480</height>
+          <format>R8G8B8</format>
+        </image>
+        <clip>
+          <near>0.05</near>
+          <far>20.0</far>
+        </clip>
+      </camera>
+    </sensor>
+  </gazebo>
+  <gazebo reference="${prefix}ee_cam_link">
+    <sensor name="${prefix}ee_cam" type="camera">
+      <pose>0 0 0 0 0 0</pose>
+      <update_rate>15</update_rate>
+      <topic>${ee_cam_topic}</topic>
+      <camera>
+        <horizontal_fov>1.3962634</horizontal_fov>
+        <image>
+          <width>640</width>
+          <height>480</height>
+          <format>R8G8B8</format>
+        </image>
+        <clip>
+          <near>0.05</near>
+          <far>20.0</far>
+        </clip>
+      </camera>
+    </sensor>
+  </gazebo>
   <xacro:if value="$(arg enable_ros2_control)">
     <xacro:if value="$(eval controllers_file != '')">
