Commit message: Agregar visual_mode y descripciones visuales para RViz
Permite separar base y brazo sin tocar TF ni controladores.

File: clean_v2/ros2_ws/src/mm_arm_description/urdf/mm_arm.urdf.xacro (robot description, xacro)
@@ -1,3 +1,4 @@
 <?xml version="1.0"?>
+<!-- Autor: Camilo Soto Villegas | Contacto: camilo.soto.v@usach.cl | Proyecto: clean_v2 -->
 <robot name="mm_arm" xmlns:xacro="http://www.ros.org/wiki/xacro">
   <xacro:include filename="$(find mm_arm_description)/urdf/mm_arm_macro.xacro"/>
@@ -7,4 +8,5 @@
   <xacro:arg name="controllers_file" default=""/>
   <xacro:arg name="enable_ros2_control" default="true"/>
+  <xacro:arg name="visual_mode" default="full"/>
   <xacro:arg name="ee_cam_mount_x" default="0.02"/>
   <xacro:arg name="ee_cam_mount_y" default="0.0"/>
@@ -26,4 +28,5 @@
     prefix="${prefix}"
     scale="${scale}"
+    visual_mode="$(arg visual_mode)"
     ee_cam_mount_x="$(arg ee_cam_mount_x)"
     ee_cam_mount_y="$(arg ee_cam_mount_y)"

File: clean_v2/ros2_ws/src/mm_arm_description/urdf/mm_arm_macro.xacro (robot description, xacro)
@@ -9,5 +9,5 @@
     </inertial>
   </xacro:macro>
-  <xacro:macro name="mm_arm" params="prefix scale ee_cam_mount_x ee_cam_mount_y ee_cam_mount_z ee_cam_mount_roll ee_cam_mount_pitch ee_cam_mount_yaw ee_cam_x ee_cam_y ee_cam_z ee_cam_roll ee_cam_pitch ee_cam_yaw">
+  <xacro:macro name="mm_arm" params="prefix scale visual_mode ee_cam_mount_x ee_cam_mount_y ee_cam_mount_z ee_cam_mount_roll ee_cam_mount_pitch ee_cam_mount_yaw ee_cam_x ee_cam_y ee_cam_z ee_cam_roll ee_cam_pitch ee_cam_yaw">
     <xacro:property name="link1_len" value="${0.22 * scale}"/>
     <xacro:property name="link2_len" value="${0.22 * scale}"/>
@@ -16,20 +16,25 @@
     <xacro:property name="link5_len" value="${0.12 * scale}"/>
     <xacro:property name="link6_len" value="${0.10 * scale}"/>
+    <xacro:property name="arm_visual_enabled" value="${visual_mode == 'full' or visual_mode == 'arm_only'}"/>
     <link name="${prefix}arm_root_link">
-      <visual>
-        <origin xyz="0 0 0.01" rpy="0 0 0"/>
-        <geometry>
-          <cylinder radius="0.05" length="0.02"/>
-        </geometry>
-      </visual>
+      <xacro:if value="${arm_visual_enabled}">
+        <visual>
+          <origin xyz="0 0 0.01" rpy="0 0 0"/>
+          <geometry>
+            <cylinder radius="0.05" length="0.02"/>
+          </geometry>
+        </visual>
+      </xacro:if>
     </link>
     <link name="${prefix}arm_base_link">
       <xacro:mm_arm_simple_inertial mass="4.0" inertia="0.02" origin_z="0.02"/>
-      <visual>
-        <origin xyz="0 0 0.02" rpy="0 0 0"/>
-        <geometry>
-          <box size="0.12 0.12 0.04"/>
-        </geometry>
-      </visual>
+      <xacro:if value="${arm_visual_enabled}">
+        <visual>
+          <origin xyz="0 0 0.02" rpy="0 0 0"/>
+          <geometry>
+            <box size="0.12 0.12 0.04"/>
+          </geometry>
+        </visual>
+      </xacro:if>
       <collision>
         <origin xyz="0 0 0.02" rpy="0 0 0"/>
@@ -46,10 +51,12 @@
     <link name="${prefix}arm_link_1">
       <xacro:mm_arm_simple_inertial mass="1.2" inertia="0.01" origin_z="${link1_len / 2.0}"/>
-      <visual>
-        <origin xyz="0 0 ${link1_len / 2.0}" rpy="0 0 0"/>
-        <geometry>
-          <box size="0.06 0.06 ${link1_len}"/>
-        </geometry>
-      </visual>
+      <xacro:if value="${arm_visual_enabled}">
+        <visual>
+          <origin xyz="0 0 ${link1_len / 2.0}" rpy="0 0 0"/>
+          <geometry>
+            <box size="0.06 0.06 ${link1_len}"/>
+          </geometry>
+        </visual>
+      </xacro:if>
       <collision>
         <origin xyz="0 0 ${link1_len / 2.0}" rpy="0 0 0"/>
@@ -68,10 +75,12 @@
     <link name="${prefix}arm_link_2">
       <xacro:mm_arm_simple_inertial mass="1.0" inertia="0.01" origin_z="${link2_len / 2.0}"/>
-      <visual>
-        <origin xyz="0 0 ${link2_len / 2.0}" rpy="0 0 0"/>
-        <geometry>
-          <box size="0.05 0.05 ${link2_len}"/>
-        </geometry>
-      </visual>
+      <xacro:if value="${arm_visual_enabled}">
+        <visual>
+          <origin xyz="0 0 ${link2_len / 2.0}" rpy="0 0 0"/>
+          <geometry>
+            <box size="0.05 0.05 ${link2_len}"/>
+          </geometry>
+        </visual>
+      </xacro:if>
       <collision>
         <origin xyz="0 0 ${link2_len / 2.0}" rpy="0 0 0"/>
@@ -90,10 +99,12 @@
     <link name="${prefix}arm_link_3">
       <xacro:mm_arm_simple_inertial mass="0.8" inertia="0.008" origin_z="${link3_len / 2.0}"/>
-      <visual>
-        <origin xyz="0 0 ${link3_len / 2.0}" rpy="0 0 0"/>
-        <geometry>
-          <box size="0.05 0.05 ${link3_len}"/>
-        </geometry>
-      </visual>
+      <xacro:if value="${arm_visual_enabled}">
+        <visual>
+          <origin xyz="0 0 ${link3_len / 2.0}" rpy="0 0 0"/>
+          <geometry>
+            <box size="0.05 0.05 ${link3_len}"/>
+          </geometry>
+        </visual>
+      </xacro:if>
       <collision>
         <origin xyz="0 0 ${link3_len / 2.0}" rpy="0 0 0"/>
@@ -112,10 +123,12 @@
     <link name="${prefix}arm_link_4">
       <xacro:mm_arm_simple_inertial mass="0.6" inertia="0.006" origin_z="${link4_len / 2.0}"/>
-      <visual>
-        <origin xyz="0 0 ${link4_len / 2.0}" rpy="0 0 0"/>
-        <geometry>
-          <box size="0.045 0.045 ${link4_len}"/>
-        </geometry>
-      </visual>
+      <xacro:if value="${arm_visual_enabled}">
+        <visual>
+          <origin xyz="0 0 ${link4_len / 2.0}" rpy="0 0 0"/>
+          <geometry>
+            <box size="0.045 0.045 ${link4_len}"/>
+          </geometry>
+        </visual>
+      </xacro:if>
       <collision>
         <origin xyz="0 0 ${link4_len / 2.0}" rpy="0 0 0"/>
@@ -134,10 +147,12 @@
     <link name="${prefix}arm_link_5">
       <xacro:mm_arm_simple_inertial mass="0.4" inertia="0.004" origin_z="${link5_len / 2.0}"/>
-      <visual>
-        <origin xyz="0 0 ${link5_len / 2.0}" rpy="0 0 0"/>
-        <geometry>
-          <box size="0.04 0.04 ${link5_len}"/>
-        </geometry>
-      </visual>
+      <xacro:if value="${arm_visual_enabled}">
+        <visual>
+          <origin xyz="0 0 ${link5_len / 2.0}" rpy="0 0 0"/>
+          <geometry>
+            <box size="0.04 0.04 ${link5_len}"/>
+          </geometry>
+        </visual>
+      </xacro:if>
       <collision>
         <origin xyz="0 0 ${link5_len / 2.0}" rpy="0 0 0"/>
@@ -156,10 +171,12 @@
     <link name="${prefix}arm_link_6">
       <xacro:mm_arm_simple_inertial mass="0.3" inertia="0.003" origin_z="${link6_len / 2.0}"/>
-      <visual>
-        <origin xyz="0 0 ${link6_len / 2.0}" rpy="0 0 0"/>
-        <geometry>
-          <box size="0.035 0.035 ${link6_len}"/>
-        </geometry>
-      </visual>
+      <xacro:if value="${arm_visual_enabled}">
+        <visual>
+          <origin xyz="0 0 ${link6_len / 2.0}" rpy="0 0 0"/>
+          <geometry>
+            <box size="0.035 0.035 ${link6_len}"/>
+          </geometry>
+        </visual>
+      </xacro:if>
       <collision>
         <origin xyz="0 0 ${link6_len / 2.0}" rpy="0 0 0"/>
@@ -177,10 +194,12 @@
     </joint>
     <link name="${prefix}tool0">
-      <visual>
-        <origin xyz="0.02 0 0" rpy="0 0 0"/>
-        <geometry>
-          <box size="0.04 0.04 0.04"/>
-        </geometry>
-      </visual>
+      <xacro:if value="${arm_visual_enabled}">
+        <visual>
+          <origin xyz="0.02 0 0" rpy="0 0 0"/>
+          <geometry>
+            <box size="0.04 0.04 0.04"/>
+          </geometry>
+        </visual>
+      </xacro:if>
     </link>
     <joint name="${prefix}tool_joint" type="fixed">
@@ -191,9 +210,11 @@
     <link name="${prefix}ee_cam_mount_link">
       <xacro:mm_arm_simple_inertial mass="0.2" inertia="0.001" origin_z="0.0"/>
-      <visual>
-        <geometry>
-          <cylinder radius="0.015" length="0.03"/>
-        </geometry>
-      </visual>
+      <xacro:if value="${arm_visual_enabled}">
+        <visual>
+          <geometry>
+            <cylinder radius="0.015" length="0.03"/>
+          </geometry>
+        </visual>
+      </xacro:if>
       <collision>
         <geometry>
@@ -209,9 +230,11 @@
     <link name="${prefix}ee_cam_link">
       <xacro:mm_arm_simple_inertial mass="0.2" inertia="0.001" origin_z="0.0"/>
-      <visual>
-        <geometry>
-          <box size="0.04 0.03 0.03"/>
-        </geometry>
-      </visual>
+      <xacro:if value="${arm_visual_enabled}">
+        <visual>
+          <geometry>
+            <box size="0.04 0.03 0.03"/>
+          </geometry>
+        </visual>
+      </xacro:if>
       <collision>
         <geometry>
@@ -227,10 +250,12 @@
     <link name="${prefix}gripper_link">
       <xacro:mm_arm_simple_inertial mass="0.2" inertia="0.0005" origin_z="0.0"/>
-      <visual>
-        <origin xyz="0.04 0 0" rpy="0 0 0"/>
-        <geometry>
-          <box size="0.08 0.02 0.02"/>
-        </geometry>
-      </visual>
+      <xacro:if value="${arm_visual_enabled}">
+        <visual>
+          <origin xyz="0.04 0 0" rpy="0 0 0"/>
+          <geometry>
+            <box size="0.08 0.02 0.02"/>
+          </geometry>
+        </visual>
+      </xacro:if>
       <collision>
         <origin xyz="0.04 0 0" rpy="0 0 0"/>

File: clean_v2/ros2_ws/src/mm_base_description/urdf/mm_base.urdf.xacro (robot description, xacro)
@@ -1,3 +1,4 @@
 <?xml version="1.0"?>
+<!-- Autor: Camilo Soto Villegas | Contacto: camilo.soto.v@usach.cl | Proyecto: clean_v2 -->
 <robot name="mm_base" xmlns:xacro="http://www.ros.org/wiki/xacro">
   <xacro:include filename="$(find mm_base_description)/urdf/mm_base_macro.xacro"/>
@@ -7,4 +8,5 @@
   <xacro:arg name="controllers_file" default=""/>
   <xacro:arg name="enable_ros2_control" default="true"/>
+  <xacro:arg name="visual_mode" default="full"/>
   <xacro:arg name="cam_front_x" default="0.26"/>
   <xacro:arg name="cam_front_y" default="0.0"/>
@@ -38,4 +40,5 @@
     prefix="${prefix}"
     scale="${scale}"
+    visual_mode="$(arg visual_mode)"
     cam_front_x="$(arg cam_front_x)"
     cam_front_y="$(arg cam_front_y)"

File: clean_v2/ros2_ws/src/mm_base_description/urdf/mm_base_macro.xacro (robot description, xacro)
@@ -9,5 +9,5 @@
     </inertial>
   </xacro:macro>
-  <xacro:macro name="mm_base" params="prefix scale cam_front_x cam_front_y cam_front_z cam_front_roll cam_front_pitch cam_front_yaw cam_left_x cam_left_y cam_left_z cam_left_roll cam_left_pitch cam_left_yaw cam_right_x cam_right_y cam_right_z cam_right_roll cam_right_pitch cam_right_yaw cam_rear_x cam_rear_y cam_rear_z cam_rear_roll cam_rear_pitch cam_rear_yaw">
+  <xacro:macro name="mm_base" params="prefix scale visual_mode cam_front_x cam_front_y cam_front_z cam_front_roll cam_front_pitch cam_front_yaw cam_left_x cam_left_y cam_left_z cam_left_roll cam_left_pitch cam_left_yaw cam_right_x cam_right_y cam_right_z cam_right_roll cam_right_pitch cam_right_yaw cam_rear_x cam_rear_y cam_rear_z cam_rear_roll cam_rear_pitch cam_rear_yaw">
     <xacro:property name="base_length" value="${0.50 * scale}"/>
     <xacro:property name="base_width" value="${0.35 * scale}"/>
@@ -19,15 +19,18 @@
     <xacro:property name="wheel_width" value="${0.04 * scale}"/>
     <link name="${prefix}base_footprint"/>
+    <xacro:property name="base_visual_enabled" value="${visual_mode == 'full' or visual_mode == 'base_only'}"/>
     <link name="${prefix}base_link">
       <xacro:mm_base_simple_inertial mass="15.0" ixz="0.25"/>
-      <visual>
-        <origin xyz="0 0 ${base_visual_height / 2.0}" rpy="0 0 0"/>
-        <geometry>
-          <box size="${base_visual_length} ${base_visual_width} ${base_visual_height}"/>
-        </geometry>
-        <material name="BaseBlue">
-          <color rgba="0.1 0.2 0.6 1.0"/>
-        </material>
-      </visual>
+      <xacro:if value="${base_visual_enabled}">
+        <visual>
+          <origin xyz="0 0 ${base_visual_height / 2.0}" rpy="0 0 0"/>
+          <geometry>
+            <box size="${base_visual_length} ${base_visual_width} ${base_visual_height}"/>
+          </geometry>
+          <material name="BaseBlue">
+            <color rgba="0.1 0.2 0.6 1.0"/>
+          </material>
+        </visual>
+      </xacro:if>
       <collision>
         <origin xyz="0 0 ${base_height / 2.0}" rpy="0 0 0"/>
@@ -44,9 +47,11 @@
     <link name="${prefix}front_left_wheel_link">
       <xacro:mm_base_simple_inertial mass="1.0" ixz="0.01"/>
-      <visual>
-        <geometry>
-          <cylinder radius="${wheel_radius}" length="${wheel_width}"/>
-        </geometry>
-      </visual>
+      <xacro:if value="${base_visual_enabled}">
+        <visual>
+          <geometry>
+            <cylinder radius="${wheel_radius}" length="${wheel_width}"/>
+          </geometry>
+        </visual>
+      </xacro:if>
       <collision>
         <geometry>
@@ -57,9 +62,11 @@
     <link name="${prefix}front_right_wheel_link">
       <xacro:mm_base_simple_inertial mass="1.0" ixz="0.01"/>
-      <visual>
-        <geometry>
-          <cylinder radius="${wheel_radius}" length="${wheel_width}"/>
-        </geometry>
-      </visual>
+      <xacro:if value="${base_visual_enabled}">
+        <visual>
+          <geometry>
+            <cylinder radius="${wheel_radius}" length="${wheel_width}"/>
+          </geometry>
+        </visual>
+      </xacro:if>
       <collision>
         <geometry>
@@ -70,9 +77,11 @@
     <link name="${prefix}rear_left_wheel_link">
       <xacro:mm_base_simple_inertial mass="1.0" ixz="0.01"/>
-      <visual>
-        <geometry>
-          <cylinder radius="${wheel_radius}" length="${wheel_width}"/>
-        </geometry>
-      </visual>
+      <xacro:if value="${base_visual_enabled}">
+        <visual>
+          <geometry>
+            <cylinder radius="${wheel_radius}" length="${wheel_width}"/>
+          </geometry>
+        </visual>
+      </xacro:if>
       <collision>
         <geometry>
@@ -83,9 +92,11 @@
     <link name="${prefix}rear_right_wheel_link">
       <xacro:mm_base_simple_inertial mass="1.0" ixz="0.01"/>
-      <visual>
-        <geometry>
-          <cylinder radius="${wheel_radius}" length="${wheel_width}"/>
-        </geometry>
-      </visual>
+      <xacro:if value="${base_visual_enabled}">
+        <visual>
+          <geometry>
+            <cylinder radius="${wheel_radius}" length="${wheel_width}"/>
+          </geometry>
+        </visual>
+      </xacro:if>
       <collision>
         <geometry>
@@ -120,9 +131,11 @@
     <link name="${prefix}cam_front_link">
       <xacro:mm_base_simple_inertial mass="0.2" ixz="0.001"/>
-      <visual>
-        <geometry>
-          <box size="0.04 0.03 0.03"/>
-        </geometry>
-      </visual>
+      <xacro:if value="${base_visual_enabled}">
+        <visual>
+          <geometry>
+            <box size="0.04 0.03 0.03"/>
+          </geometry>
+        </visual>
+      </xacro:if>
       <collision>
         <geometry>
@@ -138,9 +151,11 @@
     <link name="${prefix}cam_left_link">
       <xacro:mm_base_simple_inertial mass="0.2" ixz="0.001"/>
-      <visual>
-        <geometry>
-          <box size="0.04 0.03 0.03"/>
-        </geometry>
-      </visual>
+      <xacro:if value="${base_visual_enabled}">
+        <visual>
+          <geometry>
+            <box size="0.04 0.03 0.03"/>
+          </geometry>
+        </visual>
+      </xacro:if>
       <collision>
         <geometry>
@@ -156,9 +171,11 @@
     <link name="${prefix}cam_right_link">
       <xacro:mm_base_simple_inertial mass="0.2" ixz="0.001"/>
-      <visual>
-        <geometry>
-          <box size="0.04 0.03 0.03"/>
-        </geometry>
-      </visual>
+      <xacro:if value="${base_visual_enabled}">
+        <visual>
+          <geometry>
+            <box size="0.04 0.03 0.03"/>
+          </geometry>
+        </visual>
+      </xacro:if>
       <collision>
         <geometry>
@@ -174,9 +191,11 @@
     <link name="${prefix}cam_rear_link">
       <xacro:mm_base_simple_inertial mass="0.2" ixz="0.001"/>
-      <visual>
-        <geometry>
-          <box size="0.04 0.03 0.03"/>
-        </geometry>
-      </visual>
+      <xacro:if value="${base_visual_enabled}">
+        <visual>
+          <geometry>
+            <box size="0.04 0.03 0.03"/>
+          </geometry>
+        </visual>
+      </xacro:if>
       <collision>
         <geometry>

File: clean_v2/ros2_ws/src/mm_robot_description/urdf/mm_robot.urdf.xacro (robot description, xacro)
@@ -9,4 +9,5 @@
   <xacro:arg name="controllers_file" default=""/>
   <xacro:arg name="enable_ros2_control" default="true"/>
+  <xacro:arg name="visual_mode" default="full"/>
   <xacro:arg name="arm_x" default="0.0"/>
   <xacro:arg name="arm_y" default="0.0"/>
@@ -59,4 +60,6 @@
   <xacro:property name="scale" value="$(arg scale)"/>
   <xacro:property name="controllers_file" value="$(arg controllers_file)"/>
+  <xacro:property name="visual_mode" value="$(arg visual_mode)"/>
+  <xacro:property name="base_visual_enabled" value="${visual_mode == 'full' or visual_mode == 'base_only'}"/>
   <xacro:property name="lidar_topic" value="$(eval '/' + namespace + '/scan' if namespace != '' else '/scan')"/>
   <xacro:property name="cam_front_topic" value="$(eval '/' + namespace + '/camera/front/image_raw' if namespace != '' else '/camera/front/image_raw')"/>
@@ -68,4 +71,5 @@
     prefix="${prefix}"
     scale="${scale}"
+    visual_mode="$(arg visual_mode)"
     cam_front_x="$(arg cam_front_x)"
     cam_front_y="$(arg cam_front_y)"
@@ -96,4 +100,5 @@
     prefix="${prefix}"
     scale="${scale}"
+    visual_mode="$(arg visual_mode)"
     ee_cam_mount_x="$(arg ee_cam_mount_x)"
     ee_cam_mount_y="$(arg ee_cam_mount_y)"
@@ -121,9 +126,11 @@
         <inertia ixx="0.0002" ixy="0" ixz="0" iyy="0.0002" iyz="0" izz="0.0002"/>
       </inertial>
-      <visual>
-        <geometry>
-          <cylinder radius="0.03" length="0.05"/>
-        </geometry>
-      </visual>
+      <xacro:if value="${base_visual_enabled}">
+        <visual>
+          <geometry>
+            <cylinder radius="0.03" length="0.05"/>
+          </geometry>
+        </visual>
+      </xacro:if>
       <collision>
         <geometry>
