Commit message: Ajustar montaje fisico y defaults de simulacion
Estabiliza offsets de base/brazo/sensores y asegura Gazebo GUI sin afectar control ni TF.

File: clean_v2/ros2_ws/src/mm_arm_description/urdf/mm_arm.urdf.xacro (robot description, xacro)
@@ -8,6 +8,7 @@
   <xacro:arg name="controllers_file" default=""/>
   <xacro:arg name="enable_ros2_control" default="true"/>
+  <xacro:arg name="arm_mount_height" default="0.02"/>
   <xacro:arg name="visual_mode" default="full"/>
-  <xacro:arg name="ee_cam_mount_x" default="0.02"/>
+  <xacro:arg name="ee_cam_mount_x" default="0.055"/>
   <xacro:arg name="ee_cam_mount_y" default="0.0"/>
   <xacro:arg name="ee_cam_mount_z" default="0.02"/>
@@ -15,7 +16,7 @@
   <xacro:arg name="ee_cam_mount_pitch" default="0.0"/>
   <xacro:arg name="ee_cam_mount_yaw" default="0.0"/>
-  <xacro:arg name="ee_cam_x" default="0.08"/>
+  <xacro:arg name="ee_cam_x" default="0.035"/>
   <xacro:arg name="ee_cam_y" default="0.0"/>
-  <xacro:arg name="ee_cam_z" default="0.02"/>
+  <xacro:arg name="ee_cam_z" default="0.0"/>
   <xacro:arg name="ee_cam_roll" default="0.0"/>
   <xacro:arg name="ee_cam_pitch" default="0.0"/>
@@ -28,4 +29,5 @@
     prefix="${prefix}"
     scale="${scale}"
+    arm_mount_height="$(arg arm_mount_height)"
     visual_mode="$(arg visual_mode)"
     ee_cam_mount_x="$(arg ee_cam_mount_x)"

File: clean_v2/ros2_ws/src/mm_arm_description/urdf/mm_arm_macro.xacro (robot description, xacro)
@@ -9,5 +9,5 @@
     </inertial>
   </xacro:macro>
-  <xacro:macro name="mm_arm" params="prefix scale visual_mode ee_cam_mount_x ee_cam_mount_y ee_cam_mount_z ee_cam_mount_roll ee_cam_mount_pitch ee_cam_mount_yaw ee_cam_x ee_cam_y ee_cam_z ee_cam_roll ee_cam_pitch ee_cam_yaw">
+  <xacro:macro name="mm_arm" params="prefix scale visual_mode arm_mount_height ee_cam_mount_x ee_cam_mount_y ee_cam_mount_z ee_cam_mount_roll ee_cam_mount_pitch ee_cam_mount_yaw ee_cam_x ee_cam_y ee_cam_z ee_cam_roll ee_cam_pitch ee_cam_yaw">
     <xacro:property name="link1_len" value="${0.22 * scale}"/>
     <xacro:property name="link2_len" value="${0.22 * scale}"/>
@@ -16,4 +16,13 @@
     <xacro:property name="link5_len" value="${0.12 * scale}"/>
     <xacro:property name="link6_len" value="${0.10 * scale}"/>
+    <xacro:property name="arm_mount_height" value="${arm_mount_height}"/>
+    <xacro:property name="tool_length" value="${0.04 * scale}"/>
+    <xacro:property name="tool_width" value="${0.04 * scale}"/>
+    <xacro:property name="tool_height" value="${0.04 * scale}"/>
+    <xacro:property name="tool_visual_x" value="${tool_length / 2.0}"/>
+    <xacro:property name="gripper_length" value="${0.08 * scale}"/>
+    <xacro:property name="gripper_width" value="${0.02 * scale}"/>
+    <xacro:property name="gripper_height" value="${0.02 * scale}"/>
+    <xacro:property name="gripper_visual_x" value="${gripper_length / 2.0}"/>
     <xacro:property name="arm_visual_enabled" value="${visual_mode == 'full' or visual_mode == 'arm_only'}"/>
     <link name="${prefix}arm_root_link">
@@ -196,7 +205,7 @@
       <xacro:if value="${arm_visual_enabled}">
         <visual>
-          <origin xyz="0.02 0 0" rpy="0 0 0"/>
-          <geometry>
-            <box size="0.04 0.04 0.04"/>
+          <origin xyz="${tool_visual_x} 0 0" rpy="0 0 0"/>
+          <geometry>
+            <box size="${tool_length} ${tool_width} ${tool_height}"/>
           </geometry>
         </visual>
@@ -252,14 +261,14 @@
       <xacro:if value="${arm_visual_enabled}">
         <visual>
-          <origin xyz="0.04 0 0" rpy="0 0 0"/>
-          <geometry>
-            <box size="0.08 0.02 0.02"/>
-          </geometry>
-        </visual>
-      </xacro:if>
-      <collision>
-        <origin xyz="0.04 0 0" rpy="0 0 0"/>
-        <geometry>
-          <box size="0.08 0.02 0.02"/>
+          <origin xyz="${gripper_visual_x} 0 0" rpy="0 0 0"/>
+          <geometry>
+            <box size="${gripper_length} ${gripper_width} ${gripper_height}"/>
+          </geometry>
+        </visual>
+      </xacro:if>
+      <collision>
+        <origin xyz="${gripper_visual_x} 0 0" rpy="0 0 0"/>
+        <geometry>
+          <box size="${gripper_length} ${gripper_width} ${gripper_height}"/>
         </geometry>
       </collision>

File: clean_v2/ros2_ws/src/mm_base_description/urdf/mm_base.urdf.xacro (robot description, xacro)
@@ -9,25 +9,25 @@
   <xacro:arg name="enable_ros2_control" default="true"/>
   <xacro:arg name="visual_mode" default="full"/>
-  <xacro:arg name="cam_front_x" default="0.26"/>
+  <xacro:arg name="cam_front_x" default="0.27"/>
   <xacro:arg name="cam_front_y" default="0.0"/>
-  <xacro:arg name="cam_front_z" default="0.12"/>
+  <xacro:arg name="cam_front_z" default="0.085"/>
   <xacro:arg name="cam_front_roll" default="0.0"/>
   <xacro:arg name="cam_front_pitch" default="0.0"/>
   <xacro:arg name="cam_front_yaw" default="0.0"/>
   <xacro:arg name="cam_left_x" default="0.0"/>
-  <xacro:arg name="cam_left_y" default="0.185"/>
-  <xacro:arg name="cam_left_z" default="0.12"/>
+  <xacro:arg name="cam_left_y" default="0.19"/>
+  <xacro:arg name="cam_left_z" default="0.085"/>
   <xacro:arg name="cam_left_roll" default="0.0"/>
   <xacro:arg name="cam_left_pitch" default="0.0"/>
   <xacro:arg name="cam_left_yaw" default="1.5708"/>
   <xacro:arg name="cam_right_x" default="0.0"/>
-  <xacro:arg name="cam_right_y" default="-0.185"/>
-  <xacro:arg name="cam_right_z" default="0.12"/>
+  <xacro:arg name="cam_right_y" default="-0.19"/>
+  <xacro:arg name="cam_right_z" default="0.085"/>
   <xacro:arg name="cam_right_roll" default="0.0"/>
   <xacro:arg name="cam_right_pitch" default="0.0"/>
   <xacro:arg name="cam_right_yaw" default="-1.5708"/>
-  <xacro:arg name="cam_rear_x" default="-0.26"/>
+  <xacro:arg name="cam_rear_x" default="-0.27"/>
   <xacro:arg name="cam_rear_y" default="0.0"/>
-  <xacro:arg name="cam_rear_z" default="0.12"/>
+  <xacro:arg name="cam_rear_z" default="0.085"/>
   <xacro:arg name="cam_rear_roll" default="0.0"/>
   <xacro:arg name="cam_rear_pitch" default="0.0"/>

File: clean_v2/ros2_ws/src/mm_base_description/urdf/mm_base_macro.xacro (robot description, xacro)
@@ -10,12 +10,22 @@
   </xacro:macro>
   <xacro:macro name="mm_base" params="prefix scale visual_mode cam_front_x cam_front_y cam_front_z cam_front_roll cam_front_pitch cam_front_yaw cam_left_x cam_left_y cam_left_z cam_left_roll cam_left_pitch cam_left_yaw cam_right_x cam_right_y cam_right_z cam_right_roll cam_right_pitch cam_right_yaw cam_rear_x cam_rear_y cam_rear_z cam_rear_roll cam_rear_pitch cam_rear_yaw">
+    <xacro:property name="wheel_radius" value="${0.07 * scale}"/>
+    <xacro:property name="wheel_width" value="${0.04 * scale}"/>
     <xacro:property name="base_length" value="${0.50 * scale}"/>
     <xacro:property name="base_width" value="${0.35 * scale}"/>
     <xacro:property name="base_height" value="${0.10 * scale}"/>
-    <xacro:property name="base_visual_length" value="${base_length - (0.02 * scale)}"/>
-    <xacro:property name="base_visual_width" value="${base_width - (0.02 * scale)}"/>
-    <xacro:property name="base_visual_height" value="${base_height - (0.01 * scale)}"/>
-    <xacro:property name="wheel_radius" value="${0.07 * scale}"/>
-    <xacro:property name="wheel_width" value="${0.04 * scale}"/>
+    <xacro:property name="base_visual_margin_xy" value="${0.02 * scale}"/>
+    <xacro:property name="base_visual_margin_z" value="${0.01 * scale}"/>
+    <xacro:property name="base_visual_length" value="${base_length - base_visual_margin_xy}"/>
+    <xacro:property name="base_visual_width" value="${base_width - base_visual_margin_xy}"/>
+    <xacro:property name="base_visual_height" value="${base_height - base_visual_margin_z}"/>
+    <xacro:property name="base_visual_z" value="${base_visual_height / 2.0}"/>
+    <xacro:property name="base_collision_z" value="${base_height / 2.0}"/>
+    <xacro:property name="base_mount_z" value="${wheel_radius}"/>
+    <xacro:property name="wheel_center_z" value="0.0"/>
+    <xacro:property name="wheel_front_x" value="${base_length / 2.0}"/>
+    <xacro:property name="wheel_rear_x" value="${-base_length / 2.0}"/>
+    <xacro:property name="wheel_left_y" value="${base_width / 2.0}"/>
+    <xacro:property name="wheel_right_y" value="${-base_width / 2.0}"/>
     <link name="${prefix}base_footprint"/>
     <xacro:property name="base_visual_enabled" value="${visual_mode == 'full' or visual_mode == 'base_only'}"/>
@@ -24,5 +34,5 @@
       <xacro:if value="${base_visual_enabled}">
         <visual>
-          <origin xyz="0 0 ${base_visual_height / 2.0}" rpy="0 0 0"/>
+          <origin xyz="0 0 ${base_visual_z}" rpy="0 0 0"/>
           <geometry>
             <box size="${base_visual_length} ${base_visual_width} ${base_visual_height}"/>
@@ -34,5 +44,5 @@
       </xacro:if>
       <collision>
-        <origin xyz="0 0 ${base_height / 2.0}" rpy="0 0 0"/>
+        <origin xyz="0 0 ${base_collision_z}" rpy="0 0 0"/>
         <geometry>
           <box size="${base_length} ${base_width} ${base_height}"/>
@@ -43,5 +53,5 @@
       <parent link="${prefix}base_footprint"/>
       <child link="${prefix}base_link"/>
-      <origin xyz="0 0 ${wheel_radius}" rpy="0 0 0"/>
+      <origin xyz="0 0 ${base_mount_z}" rpy="0 0 0"/>
     </joint>
     <link name="${prefix}front_left_wheel_link">
@@ -108,5 +118,5 @@
       <parent link="${prefix}base_link"/>
       <child link="${prefix}front_left_wheel_link"/>
-      <origin xyz="${base_length / 2.0} ${base_width / 2.0} 0.0" rpy="0 1.5708 0"/>
+      <origin xyz="${wheel_front_x} ${wheel_left_y} ${wheel_center_z}" rpy="0 1.5708 0"/>
       <axis xyz="0 0 1"/>
     </joint>
@@ -114,5 +124,5 @@
       <parent link="${prefix}base_link"/>
       <child link="${prefix}front_right_wheel_link"/>
-      <origin xyz="${base_length / 2.0} -${base_width / 2.0} 0.0" rpy="0 1.5708 0"/>
+      <origin xyz="${wheel_front_x} ${wheel_right_y} ${wheel_center_z}" rpy="0 1.5708 0"/>
       <axis xyz="0 0 1"/>
     </joint>
@@ -120,5 +130,5 @@
       <parent link="${prefix}base_link"/>
       <child link="${prefix}rear_left_wheel_link"/>
-      <origin xyz="-${base_length / 2.0} ${base_width / 2.0} 0.0" rpy="0 1.5708 0"/>
+      <origin xyz="${wheel_rear_x} ${wheel_left_y} ${wheel_center_z}" rpy="0 1.5708 0"/>
       <axis xyz="0 0 1"/>
     </joint>
@@ -126,5 +136,5 @@
       <parent link="${prefix}base_link"/>
       <child link="${prefix}rear_right_wheel_link"/>
-      <origin xyz="-${base_length / 2.0} -${base_width / 2.0} 0.0" rpy="0 1.5708 0"/>
+      <origin xyz="${wheel_rear_x} ${wheel_right_y} ${wheel_center_z}" rpy="0 1.5708 0"/>
       <axis xyz="0 0 1"/>
     </joint>

File: clean_v2/ros2_ws/src/mm_robot_description/urdf/mm_robot.urdf.xacro (robot description, xacro)
@@ -12,5 +12,5 @@
   <xacro:arg name="arm_x" default="0.0"/>
   <xacro:arg name="arm_y" default="0.0"/>
-  <xacro:arg name="arm_z" default="0.05"/>
+  <xacro:arg name="arm_z" default="0.015"/>
   <xacro:arg name="arm_roll" default="0.0"/>
   <xacro:arg name="arm_pitch" default="0.0"/>
@@ -19,30 +19,30 @@
   <xacro:arg name="lidar_x" default="0.20"/>
   <xacro:arg name="lidar_y" default="0.0"/>
-  <xacro:arg name="lidar_z" default="0.15"/>
-  <xacro:arg name="cam_front_x" default="0.26"/>
+  <xacro:arg name="lidar_z" default="0.125"/>
+  <xacro:arg name="cam_front_x" default="0.27"/>
   <xacro:arg name="cam_front_y" default="0.0"/>
-  <xacro:arg name="cam_front_z" default="0.12"/>
+  <xacro:arg name="cam_front_z" default="0.085"/>
   <xacro:arg name="cam_front_roll" default="0.0"/>
   <xacro:arg name="cam_front_pitch" default="0.0"/>
   <xacro:arg name="cam_front_yaw" default="0.0"/>
   <xacro:arg name="cam_left_x" default="0.0"/>
-  <xacro:arg name="cam_left_y" default="0.185"/>
-  <xacro:arg name="cam_left_z" default="0.12"/>
+  <xacro:arg name="cam_left_y" default="0.19"/>
+  <xacro:arg name="cam_left_z" default="0.085"/>
   <xacro:arg name="cam_left_roll" default="0.0"/>
   <xacro:arg name="cam_left_pitch" default="0.0"/>
   <xacro:arg name="cam_left_yaw" default="1.5708"/>
   <xacro:arg name="cam_right_x" default="0.0"/>
-  <xacro:arg name="cam_right_y" default="-0.185"/>
-  <xacro:arg name="cam_right_z" default="0.12"/>
+  <xacro:arg name="cam_right_y" default="-0.19"/>
+  <xacro:arg name="cam_right_z" default="0.085"/>
   <xacro:arg name="cam_right_roll" default="0.0"/>
   <xacro:arg name="cam_right_pitch" default="0.0"/>
   <xacro:arg name="cam_right_yaw" default="-1.5708"/>
-  <xacro:arg name="cam_rear_x" default="-0.26"/>
+  <xacro:arg name="cam_rear_x" default="-0.27"/>
   <xacro:arg name="cam_rear_y" default="0.0"/>
-  <xacro:arg name="cam_rear_z" default="0.12"/>
+  <xacro:arg name="cam_rear_z" default="0.085"/>
   <xacro:arg name="cam_rear_roll" default="0.0"/>
   <xacro:arg name="cam_rear_pitch" default="0.0"/>
   <xacro:arg name="cam_rear_yaw" default="3.1416"/>
-  <xacro:arg name="ee_cam_mount_x" default="0.02"/>
+  <xacro:arg name="ee_cam_mount_x" default="0.055"/>
   <xacro:arg name="ee_cam_mount_y" default="0.0"/>
   <xacro:arg name="ee_cam_mount_z" default="0.02"/>
@@ -50,7 +50,7 @@
   <xacro:arg name="ee_cam_mount_pitch" default="0.0"/>
   <xacro:arg name="ee_cam_mount_yaw" default="0.0"/>
-  <xacro:arg name="ee_cam_x" default="0.08"/>
+  <xacro:arg name="ee_cam_x" default="0.035"/>
   <xacro:arg name="ee_cam_y" default="0.0"/>
-  <xacro:arg name="ee_cam_z" default="0.02"/>
+  <xacro:arg name="ee_cam_z" default="0.0"/>
   <xacro:arg name="ee_cam_roll" default="0.0"/>
   <xacro:arg name="ee_cam_pitch" default="0.0"/>
@@ -61,4 +61,7 @@
   <xacro:property name="controllers_file" value="$(arg controllers_file)"/>
   <xacro:property name="visual_mode" value="$(arg visual_mode)"/>
+  <xacro:property name="base_height" value="${0.10 * scale}"/>
+  <xacro:property name="arm_mount_height" value="$(arg arm_z)"/>
+  <xacro:property name="arm_mount_z" value="${base_height + arm_mount_height}"/>
   <xacro:property name="base_visual_enabled" value="${visual_mode == 'full' or visual_mode == 'base_only'}"/>
   <xacro:property name="lidar_topic" value="$(eval '/' + namespace + '/scan' if namespace != '' else '/scan')"/>
@@ -100,4 +103,5 @@
     prefix="${prefix}"
     scale="${scale}"
+    arm_mount_height="${arm_mount_height}"
     visual_mode="$(arg visual_mode)"
     ee_cam_mount_x="$(arg ee_cam_mount_x)"
@@ -117,5 +121,5 @@
     <parent link="${prefix}base_link"/>
     <child link="${prefix}arm_root_link"/>
-    <origin xyz="$(arg arm_x) $(arg arm_y) $(arg arm_z)" rpy="$(arg arm_roll) $(arg arm_pitch) $(arg arm_yaw)"/>
+    <origin xyz="$(arg arm_x) $(arg arm_y) ${arm_mount_z}" rpy="$(arg arm_roll) $(arg arm_pitch) $(arg arm_yaw)"/>
   </joint>
   <xacro:if value="$(arg enable_lidar)">

Commit message: feat(sim): agregar IMU en efector final y bridge namespaced

File: clean_v2/ros2_ws/src/mm_arm_description/urdf/mm_arm.urdf.xacro (robot description, xacro)
@@ -22,4 +22,11 @@
   <xacro:arg name="ee_cam_pitch" default="0.0"/>
   <xacro:arg name="ee_cam_yaw" default="0.0"/>
+  <xacro:arg name="enable_ee_imu" default="true"/>
+  <xacro:arg name="ee_imu_x" default="0.03"/>
+  <xacro:arg name="ee_imu_y" default="0.0"/>
+  <xacro:arg name="ee_imu_z" default="0.02"/>
+  <xacro:arg name="ee_imu_roll" default="0.0"/>
+  <xacro:arg name="ee_imu_pitch" default="0.0"/>
+  <xacro:arg name="ee_imu_yaw" default="0.0"/>
   <xacro:property name="prefix" value="$(arg prefix)"/>
   <xacro:property name="namespace" value="$(arg namespace)"/>
@@ -43,4 +50,11 @@
     ee_cam_pitch="$(arg ee_cam_pitch)"
     ee_cam_yaw="$(arg ee_cam_yaw)"
+    enable_ee_imu="$(arg enable_ee_imu)"
+    ee_imu_x="$(arg ee_imu_x)"
+    ee_imu_y="$(arg ee_imu_y)"
+    ee_imu_z="$(arg ee_imu_z)"
+    ee_imu_roll="$(arg ee_imu_roll)"
+    ee_imu_pitch="$(arg ee_imu_pitch)"
+    ee_imu_yaw="$(arg ee_imu_yaw)"
   />
   <xacro:if value="$(arg enable_ros2_control)">

File: clean_v2/ros2_ws/src/mm_arm_description/urdf/mm_arm_macro.xacro (robot description, xacro)
@@ -9,5 +9,5 @@
     </inertial>
   </xacro:macro>
-  <xacro:macro name="mm_arm" params="prefix scale visual_mode arm_mount_height ee_cam_mount_x ee_cam_mount_y ee_cam_mount_z ee_cam_mount_roll ee_cam_mount_pitch ee_cam_mount_yaw ee_cam_x ee_cam_y ee_cam_z ee_cam_roll ee_cam_pitch ee_cam_yaw">
+  <xacro:macro name="mm_arm" params="prefix scale visual_mode arm_mount_height ee_cam_mount_x ee_cam_mount_y ee_cam_mount_z ee_cam_mount_roll ee_cam_mount_pitch ee_cam_mount_yaw ee_cam_x ee_cam_y ee_cam_z ee_cam_roll ee_cam_pitch ee_cam_yaw enable_ee_imu ee_imu_x ee_imu_y ee_imu_z ee_imu_roll ee_imu_pitch ee_imu_yaw">
     <xacro:property name="link1_len" value="${0.22 * scale}"/>
     <xacro:property name="link2_len" value="${0.22 * scale}"/>
@@ -257,4 +257,26 @@
       <origin xyz="${ee_cam_x} ${ee_cam_y} ${ee_cam_z}" rpy="${ee_cam_roll} ${ee_cam_pitch} ${ee_cam_yaw}"/>
     </joint>
+    <xacro:if value="${enable_ee_imu}">
+      <link name="${prefix}ee_imu_link">
+        <xacro:mm_arm_simple_inertial mass="0.1" inertia="0.0002" origin_z="0.0"/>
+        <xacro:if value="${arm_visual_enabled}">
+          <visual>
+            <geometry>
+              <box size="0.03 0.03 0.02"/>
+            </geometry>
+          </visual>
+        </xacro:if>
+        <collision>
+          <geometry>
+            <box size="0.03 0.03 0.02"/>
+          </geometry>
+        </collision>
+      </link>
+      <joint name="${prefix}ee_imu_joint" type="fixed">
+        <parent link="${prefix}tool0"/>
+        <child link="${prefix}ee_imu_link"/>
+        <origin xyz="${ee_imu_x} ${ee_imu_y} ${ee_imu_z}" rpy="${ee_imu_roll} ${ee_imu_pitch} ${ee_imu_yaw}"/>
+      </joint>
+    </xacro:if>
     <link name="${prefix}gripper_link">
       <xacro:mm_arm_simple_inertial mass="0.2" inertia="0.0005" origin_z="0.0"/>

File: clean_v2/ros2_ws/src/mm_robot_description/urdf/mm_robot.urdf.xacro (robot description, xacro)
@@ -60,4 +60,11 @@
   <xacro:arg name="imu_y" default="0.0"/>
   <xacro:arg name="imu_z" default="0.10"/>
+  <xacro:arg name="enable_ee_imu" default="true"/>
+  <xacro:arg name="ee_imu_x" default="0.03"/>
+  <xacro:arg name="ee_imu_y" default="0.0"/>
+  <xacro:arg name="ee_imu_z" default="0.02"/>
+  <xacro:arg name="ee_imu_roll" default="0.0"/>
+  <xacro:arg name="ee_imu_pitch" default="0.0"/>
+  <xacro:arg name="ee_imu_yaw" default="0.0"/>
   <xacro:property name="prefix" value="$(arg prefix)"/>
   <xacro:property name="namespace" value="$(arg namespace)"/>
@@ -75,4 +82,5 @@
   <xacro:property name="cam_rear_topic" value="$(eval '/' + namespace + '/camera/rear/image_raw' if namespace != '' else '/camera/rear/image_raw')"/>
   <xacro:property name="ee_cam_topic" value="$(eval '/' + namespace + '/camera/ee/image_raw' if namespace != '' else '/camera/ee/image_raw')"/>
+  <xacro:property name="ee_imu_topic" value="$(eval '/' + namespace + '/imu/ee_raw' if namespace != '' else '/imu/ee_raw')"/>
   <xacro:mm_base
     prefix="${prefix}"
@@ -121,4 +129,11 @@
     ee_cam_pitch="$(arg ee_cam_pitch)"
     ee_cam_yaw="$(arg ee_cam_yaw)"
+    enable_ee_imu="$(arg enable_ee_imu)"
+    ee_imu_x="$(arg ee_imu_x)"
+    ee_imu_y="$(arg ee_imu_y)"
+    ee_imu_z="$(arg ee_imu_z)"
+    ee_imu_roll="$(arg ee_imu_roll)"
+    ee_imu_pitch="$(arg ee_imu_pitch)"
+    ee_imu_yaw="$(arg ee_imu_yaw)"
   />
   <joint name="${prefix}base_to_arm_joint" type="fixed">
@@ -216,4 +231,57 @@
         <update_rate>100</update_rate>
         <topic>$(eval '/' + namespace + '/imu_raw' if namespace != '' else '/imu_raw')</topic>
+        <imu>
+          <linear_acceleration>
+            <x>
+              <noise type="gaussian">
+                <mean>0.0</mean>
+                <stddev>0.01</stddev>
+              </noise>
+            </x>
+            <y>
+              <noise type="gaussian">
+                <mean>0.0</mean>
+                <stddev>0.01</stddev>
+              </noise>
+            </y>
+            <z>
+              <noise type="gaussian">
+                <mean>0.0</mean>
+                <stddev>0.01</stddev>
+              </noise>
+            </z>
+          </linear_acceleration>
+          <angular_velocity>
+            <x>
+              <noise type="gaussian">
+                <mean>0.0</mean>
+                <stddev>0.001</stddev>
+              </noise>
+            </x>
+            <y>
+              <noise type="gaussian">
+                <mean>0.0</mean>
+                <stddev>0.001</stddev>
+              </noise>
+            </y>
+            <z>
+              <noise type="gaussian">
+                <mean>0.0</mean>
+                <stddev>0.001</stddev>
+              </noise>
+            </z>
+          </angular_velocity>
+        </imu>
+      </sensor>
+    </gazebo>
+  </xacro:if>
+  <!-- IMU Sensor on end-effector link -->
+  <xacro:if value="$(arg enable_ee_imu)">
+    <gazebo reference="${prefix}ee_imu_link">
+      <sensor name="${prefix}ee_imu" type="imu">
+        <pose>0 0 0 0 0 0</pose>
+        <always_on>1</always_on>
+        <update_rate>100</update_rate>
+        <topic>${ee_imu_topic}</topic>
         <imu>
           <linear_acceleration>
