Commit message: fix(sim): corregir parámetros físicos basados en mejores prácticas
- Inercias corregidas con fórmulas físicamente correctas:
  * mm_base_macro.xacro: box_inertial para base/cámaras, cylinder_inertial_y para ruedas
  * mm_arm_macro.xacro: box_inertial y cylinder_inertial_z según geometrías

- Controlador omnidireccional corregido:
  * robot_radius: 0.305 → 0.357m (cálculo geométrico correcto)
  * wheel_offset: 0.611 → 0.742 rad (ángulo correcto de primera rueda)

- Nav2 configurado para robot omnidireccional rectangular:
  * Footprint agregado en global/local costmap [[0.25, 0.30], [0.25, -0.30], [-0.25, -0.30], [-0.25, 0.30]]
  * AMCL con OmnidirectionalMotionModel y parámetros alpha3=0.3, alpha5=0.3

- MoveIt kinematics optimizado para brazo 6-DOF:
  * timeout: 0.1s → 0.5s
  * attempts: 3 → 10

Basado en: docs/BEST_PRACTICES_FROM_PUBLIC_REPOS.md

Co-Authored-By: Claude Sonnet 4.5 <noreply@anthropic.com>

File: clean_v2/ros2_ws/src/mm_arm_description/urdf/mm_arm_macro.xacro (robot description, xacro)
@@ -2,9 +2,24 @@
 <!-- Autor: Camilo Soto Villegas | Contacto: camilo.soto.v@usach.cl | Proyecto: clean_v2 -->
 <robot xmlns:xacro="http://www.ros.org/wiki/xacro">
-  <xacro:macro name="mm_arm_simple_inertial" params="mass inertia origin_z">
+  <!-- Macro para inercia de caja (box) -->
+  <xacro:macro name="box_inertial" params="mass x y z *origin">
     <inertial>
-      <origin xyz="0 0 ${origin_z}" rpy="0 0 0"/>
+      <xacro:insert_block name="origin"/>
       <mass value="${mass}"/>
-      <inertia ixx="${inertia}" ixy="0" ixz="0" iyy="${inertia}" iyz="0" izz="${inertia}"/>
+      <inertia
+        ixx="${(mass/12) * (y*y + z*z)}" ixy="0.0" ixz="0.0"
+        iyy="${(mass/12) * (x*x + z*z)}" iyz="0.0"
+        izz="${(mass/12) * (x*x + y*y)}"/>
+    </inertial>
+  </xacro:macro>
+  <!-- Macro para inercia de cilindro alineado con eje Z -->
+  <xacro:macro name="cylinder_inertial_z" params="mass radius length *origin">
+    <inertial>
+      <xacro:insert_block name="origin"/>
+      <mass value="${mass}"/>
+      <inertia
+        ixx="${(mass/12) * (3*radius*radius + length*length)}" ixy="0.0" ixz="0.0"
+        iyy="${(mass/12) * (3*radius*radius + length*length)}" iyz="0.0"
+        izz="${0.5 * mass * radius * radius}"/>
     </inertial>
   </xacro:macro>
@@ -37,5 +52,7 @@
     </link>
     <link name="${prefix}arm_base_link">
-      <xacro:mm_arm_simple_inertial mass="4.0" inertia="0.02" origin_z="0.02"/>
+      <xacro:box_inertial mass="4.0" x="0.12" y="0.12" z="0.04">
+        <origin xyz="0 0 0.02" rpy="0 0 0"/>
+      </xacro:box_inertial>
       <xacro:if value="${arm_visual_enabled}">
         <visual>
@@ -59,5 +76,7 @@
     </joint>
     <link name="${prefix}arm_link_1">
-      <xacro:mm_arm_simple_inertial mass="1.2" inertia="0.01" origin_z="${link1_len / 2.0}"/>
+      <xacro:box_inertial mass="1.2" x="0.06" y="0.06" z="${link1_len}">
+        <origin xyz="0 0 ${link1_len / 2.0}" rpy="0 0 0"/>
+      </xacro:box_inertial>
       <xacro:if value="${arm_visual_enabled}">
         <visual>
@@ -83,5 +102,7 @@
     </joint>
     <link name="${prefix}arm_link_2">
-      <xacro:mm_arm_simple_inertial mass="1.0" inertia="0.01" origin_z="${link2_len / 2.0}"/>
+      <xacro:box_inertial mass="1.0" x="0.05" y="0.05" z="${link2_len}">
+        <origin xyz="0 0 ${link2_len / 2.0}" rpy="0 0 0"/>
+      </xacro:box_inertial>
       <xacro:if value="${arm_visual_enabled}">
         <visual>
@@ -107,5 +128,7 @@
     </joint>
     <link name="${prefix}arm_link_3">
-      <xacro:mm_arm_simple_inertial mass="0.8" inertia="0.008" origin_z="${link3_len / 2.0}"/>
+      <xacro:box_inertial mass="0.8" x="0.05" y="0.05" z="${link3_len}">
+        <origin xyz="0 0 ${link3_len / 2.0}" rpy="0 0 0"/>
+      </xacro:box_inertial>
       <xacro:if value="${arm_visual_enabled}">
         <visual>
@@ -131,5 +154,7 @@
     </joint>
     <link name="${prefix}arm_link_4">
-      <xacro:mm_arm_simple_inertial mass="0.6" inertia="0.006" origin_z="${link4_len / 2.0}"/>
+      <xacro:box_inertial mass="0.6" x="0.045" y="0.045" z="${link4_len}">
+        <origin xyz="0 0 ${link4_len / 2.0}" rpy="0 0 0"/>
+      </xacro:box_inertial>
       <xacro:if value="${arm_visual_enabled}">
         <visual>
@@ -155,5 +180,7 @@
     </joint>
     <link name="${prefix}arm_link_5">
-      <xacro:mm_arm_simple_inertial mass="0.4" inertia="0.004" origin_z="${link5_len / 2.0}"/>
+      <xacro:box_inertial mass="0.4" x="0.04" y="0.04" z="${link5_len}">
+        <origin xyz="0 0 ${link5_len / 2.0}" rpy="0 0 0"/>
+      </xacro:box_inertial>
       <xacro:if value="${arm_visual_enabled}">
         <visual>
@@ -179,5 +206,7 @@
     </joint>
     <link name="${prefix}arm_link_6">
-      <xacro:mm_arm_simple_inertial mass="0.3" inertia="0.003" origin_z="${link6_len / 2.0}"/>
+      <xacro:box_inertial mass="0.3" x="0.035" y="0.035" z="${link6_len}">
+        <origin xyz="0 0 ${link6_len / 2.0}" rpy="0 0 0"/>
+      </xacro:box_inertial>
       <xacro:if value="${arm_visual_enabled}">
         <visual>
@@ -218,5 +247,7 @@
     </joint>
     <link name="${prefix}ee_cam_mount_link">
-      <xacro:mm_arm_simple_inertial mass="0.2" inertia="0.001" origin_z="0.0"/>
+      <xacro:cylinder_inertial_z mass="0.2" radius="0.015" length="0.03">
+        <origin xyz="0 0 0" rpy="0 0 0"/>
+      </xacro:cylinder_inertial_z>
       <xacro:if value="${arm_visual_enabled}">
         <visual>
@@ -238,5 +269,7 @@
     </joint>
     <link name="${prefix}ee_cam_link">
-      <xacro:mm_arm_simple_inertial mass="0.2" inertia="0.001" origin_z="0.0"/>
+      <xacro:box_inertial mass="0.2" x="0.04" y="0.03" z="0.03">
+        <origin xyz="0 0 0" rpy="0 0 0"/>
+      </xacro:box_inertial>
       <xacro:if value="${arm_visual_enabled}">
         <visual>
@@ -259,5 +292,7 @@
     <xacro:if value="${enable_ee_imu}">
       <link name="${prefix}ee_imu_link">
-        <xacro:mm_arm_simple_inertial mass="0.1" inertia="0.0002" origin_z="0.0"/>
+        <xacro:box_inertial mass="0.1" x="0.03" y="0.03" z="0.02">
+          <origin xyz="0 0 0" rpy="0 0 0"/>
+        </xacro:box_inertial>
         <xacro:if value="${arm_visual_enabled}">
           <visual>
@@ -280,5 +315,7 @@
     </xacro:if>
     <link name="${prefix}gripper_link">
-      <xacro:mm_arm_simple_inertial mass="0.2" inertia="0.0005" origin_z="0.0"/>
+      <xacro:box_inertial mass="0.2" x="${gripper_length}" y="${gripper_width}" z="${gripper_height}">
+        <origin xyz="0 0 0" rpy="0 0 0"/>
+      </xacro:box_inertial>
       <xacro:if value="${arm_visual_enabled}">
         <visual>

File: clean_v2/ros2_ws/src/mm_base_description/urdf/mm_base_macro.xacro (robot description, xacro)
@@ -2,9 +2,24 @@
 <!-- Autor: Camilo Soto Villegas | Contacto: camilo.soto.v@usach.cl | Proyecto: clean_v2 -->
 <robot xmlns:xacro="http://www.ros.org/wiki/xacro">
-  <xacro:macro name="mm_base_simple_inertial" params="mass ixz">
+  <!-- Macro para inercia de caja (box) -->
+  <xacro:macro name="box_inertial" params="mass x y z *origin">
     <inertial>
-      <origin xyz="0 0 0" rpy="0 0 0"/>
+      <xacro:insert_block name="origin"/>
       <mass value="${mass}"/>
-      <inertia ixx="${ixz}" ixy="0" ixz="0" iyy="${ixz}" iyz="0" izz="${ixz}"/>
+      <inertia
+        ixx="${(mass/12) * (y*y + z*z)}" ixy="0.0" ixz="0.0"
+        iyy="${(mass/12) * (x*x + z*z)}" iyz="0.0"
+        izz="${(mass/12) * (x*x + y*y)}"/>
+    </inertial>
+  </xacro:macro>
+  <!-- Macro para inercia de cilindro alineado con eje Y (ruedas) -->
+  <xacro:macro name="cylinder_inertial_y" params="mass radius length *origin">
+    <inertial>
+      <xacro:insert_block name="origin"/>
+      <mass value="${mass}"/>
+      <inertia
+        ixx="${(mass/12) * (3*radius*radius + length*length)}" ixy="0.0" ixz="0.0"
+        iyy="${0.5 * mass * radius * radius}" iyz="0.0"
+        izz="${(mass/12) * (3*radius*radius + length*length)}"/>
     </inertial>
   </xacro:macro>
@@ -31,5 +46,7 @@
     <xacro:property name="base_visual_enabled" value="${visual_mode == 'full' or visual_mode == 'base_only'}"/>
     <link name="${prefix}base_link">
-      <xacro:mm_base_simple_inertial mass="15.0" ixz="0.25"/>
+      <xacro:box_inertial mass="15.0" x="${base_length}" y="${base_width}" z="${base_height}">
+        <origin xyz="0 0 0" rpy="0 0 0"/>
+      </xacro:box_inertial>
       <xacro:if value="${base_visual_enabled}">
         <visual>
@@ -56,5 +73,7 @@
     </joint>
     <link name="${prefix}front_left_wheel_link">
-      <xacro:mm_base_simple_inertial mass="1.0" ixz="0.01"/>
+      <xacro:cylinder_inertial_y mass="1.0" radius="${wheel_radius}" length="${wheel_width}">
+        <origin xyz="0 0 0" rpy="0 0 0"/>
+      </xacro:cylinder_inertial_y>
       <xacro:if value="${base_visual_enabled}">
         <visual>
@@ -71,5 +90,7 @@
     </link>
     <link name="${prefix}front_right_wheel_link">
-      <xacro:mm_base_simple_inertial mass="1.0" ixz="0.01"/>
+      <xacro:cylinder_inertial_y mass="1.0" radius="${wheel_radius}" length="${wheel_width}">
+        <origin xyz="0 0 0" rpy="0 0 0"/>
+      </xacro:cylinder_inertial_y>
       <xacro:if value="${base_visual_enabled}">
         <visual>
@@ -86,5 +107,7 @@
     </link>
     <link name="${prefix}rear_left_wheel_link">
-      <xacro:mm_base_simple_inertial mass="1.0" ixz="0.01"/>
+      <xacro:cylinder_inertial_y mass="1.0" radius="${wheel_radius}" length="${wheel_width}">
+        <origin xyz="0 0 0" rpy="0 0 0"/>
+      </xacro:cylinder_inertial_y>
       <xacro:if value="${base_visual_enabled}">
         <visual>
@@ -101,5 +124,7 @@
     </link>
     <link name="${prefix}rear_right_wheel_link">
-      <xacro:mm_base_simple_inertial mass="1.0" ixz="0.01"/>
+      <xacro:cylinder_inertial_y mass="1.0" radius="${wheel_radius}" length="${wheel_width}">
+        <origin xyz="0 0 0" rpy="0 0 0"/>
+      </xacro:cylinder_inertial_y>
       <xacro:if value="${base_visual_enabled}">
         <visual>
@@ -140,5 +165,7 @@
     </joint>
     <link name="${prefix}cam_front_link">
-      <xacro:mm_base_simple_inertial mass="0.2" ixz="0.001"/>
+      <xacro:box_inertial mass="0.2" x="0.04" y="0.03" z="0.03">
+        <origin xyz="0 0 0" rpy="0 0 0"/>
+      </xacro:box_inertial>
       <xacro:if value="${base_visual_enabled}">
         <visual>
@@ -160,5 +187,7 @@
     </joint>
     <link name="${prefix}cam_left_link">
-      <xacro:mm_base_simple_inertial mass="0.2" ixz="0.001"/>
+      <xacro:box_inertial mass="0.2" x="0.04" y="0.03" z="0.03">
+        <origin xyz="0 0 0" rpy="0 0 0"/>
+      </xacro:box_inertial>
       <xacro:if value="${base_visual_enabled}">
         <visual>
@@ -180,5 +209,7 @@
     </joint>
     <link name="${prefix}cam_right_link">
-      <xacro:mm_base_simple_inertial mass="0.2" ixz="0.001"/>
+      <xacro:box_inertial mass="0.2" x="0.04" y="0.03" z="0.03">
+        <origin xyz="0 0 0" rpy="0 0 0"/>
+      </xacro:box_inertial>
       <xacro:if value="${base_visual_enabled}">
         <visual>
@@ -200,5 +231,7 @@
     </joint>
     <link name="${prefix}cam_rear_link">
-      <xacro:mm_base_simple_inertial mass="0.2" ixz="0.001"/>
+      <xacro:box_inertial mass="0.2" x="0.04" y="0.03" z="0.03">
+        <origin xyz="0 0 0" rpy="0 0 0"/>
+      </xacro:box_inertial>
       <xacro:if value="${base_visual_enabled}">
         <visual>
