Commit message: Simplify visuals and align metadata headers

File: clean_v2/ros2_ws/src/mm_arm_description/urdf/mm_arm_macro.xacro (robot description, xacro)
@@ -1,3 +1,4 @@
 <?xml version="1.0"?>
+<!-- Autor: Camilo Soto Villegas | Contacto: camilo.soto.v@usach.cl | Proyecto: clean_v2 -->
 <robot xmlns:xacro="http://www.ros.org/wiki/xacro">
   <xacro:macro name="mm_arm_simple_inertial" params="mass inertia origin_z">
@@ -15,5 +16,12 @@
     <xacro:property name="link5_len" value="${0.12 * scale}"/>
     <xacro:property name="link6_len" value="${0.10 * scale}"/>
-    <link name="${prefix}arm_root_link"/>
+    <link name="${prefix}arm_root_link">
+      <visual>
+        <origin xyz="0 0 0.01" rpy="0 0 0"/>
+        <geometry>
+          <cylinder radius="0.05" length="0.02"/>
+        </geometry>
+      </visual>
+    </link>
     <link name="${prefix}arm_base_link">
       <xacro:mm_arm_simple_inertial mass="4.0" inertia="0.02" origin_z="0.02"/>
@@ -168,5 +176,12 @@
       <limit lower="-3.14" upper="3.14" effort="10" velocity="2.0"/>
     </joint>
-    <link name="${prefix}tool0"/>
+    <link name="${prefix}tool0">
+      <visual>
+        <origin xyz="0.02 0 0" rpy="0 0 0"/>
+        <geometry>
+          <box size="0.04 0.04 0.04"/>
+        </geometry>
+      </visual>
+    </link>
     <joint name="${prefix}tool_joint" type="fixed">
       <parent link="${prefix}arm_link_6"/>

File: clean_v2/ros2_ws/src/mm_base_description/urdf/mm_base_macro.xacro (robot description, xacro)
@@ -1,3 +1,4 @@
 <?xml version="1.0"?>
+<!-- Autor: Camilo Soto Villegas | Contacto: camilo.soto.v@usach.cl | Proyecto: clean_v2 -->
 <robot xmlns:xacro="http://www.ros.org/wiki/xacro">
   <xacro:macro name="mm_base_simple_inertial" params="mass ixz">
@@ -12,4 +13,7 @@
     <xacro:property name="base_width" value="${0.35 * scale}"/>
     <xacro:property name="base_height" value="${0.10 * scale}"/>
+    <xacro:property name="base_visual_length" value="${base_length - (0.02 * scale)}"/>
+    <xacro:property name="base_visual_width" value="${base_width - (0.02 * scale)}"/>
+    <xacro:property name="base_visual_height" value="${base_height - (0.01 * scale)}"/>
     <xacro:property name="wheel_radius" value="${0.07 * scale}"/>
     <xacro:property name="wheel_width" value="${0.04 * scale}"/>
@@ -18,7 +22,7 @@
       <xacro:mm_base_simple_inertial mass="15.0" ixz="0.25"/>
       <visual>
-        <origin xyz="0 0 ${base_height / 2.0}" rpy="0 0 0"/>
+        <origin xyz="0 0 ${base_visual_height / 2.0}" rpy="0 0 0"/>
         <geometry>
-          <box size="${base_length} ${base_width} ${base_height}"/>
+          <box size="${base_visual_length} ${base_visual_width} ${base_visual_height}"/>
         </geometry>
         <material name="BaseBlue">

File: clean_v2/ros2_ws/src/mm_robot_description/urdf/mm_robot.urdf.xacro (robot description, xacro)
@@ -1,3 +1,4 @@
 <?xml version="1.0"?>
+<!-- Autor: Camilo Soto Villegas | Contacto: camilo.soto.v@usach.cl | Proyecto: clean_v2 -->
 <robot name="mm_mobile_manipulator" xmlns:xacro="http://www.ros.org/wiki/xacro">
   <xacro:include filename="$(find mm_base_description)/urdf/mm_base_macro.xacro"/>

Commit message: fix(sim): dedupe ee imu and pass topic to arm macro

File: clean_v2/ros2_ws/src/mm_arm_description/urdf/mm_arm_macro.xacro (robot description, xacro)
@@ -24,5 +24,5 @@
     </inertial>
   </xacro:macro>
-  <xacro:macro name="mm_arm" params="prefix scale visual_mode arm_mount_height ee_cam_mount_x ee_cam_mount_y ee_cam_mount_z ee_cam_mount_roll ee_cam_mount_pitch ee_cam_mount_yaw ee_cam_x ee_cam_y ee_cam_z ee_cam_roll ee_cam_pitch ee_cam_yaw enable_ee_imu ee_imu_x ee_imu_y ee_imu_z ee_imu_roll ee_imu_pitch ee_imu_yaw">
+  <xacro:macro name="mm_arm" params="prefix scale visual_mode arm_mount_height ee_cam_mount_x ee_cam_mount_y ee_cam_mount_z ee_cam_mount_roll ee_cam_mount_pitch ee_cam_mount_yaw ee_cam_x ee_cam_y ee_cam_z ee_cam_roll ee_cam_pitch ee_cam_yaw enable_ee_imu ee_imu_x ee_imu_y ee_imu_z ee_imu_roll ee_imu_pitch ee_imu_yaw ee_imu_topic">
     <xacro:property name="link1_len" value="${0.22 * scale}"/>
     <xacro:property name="link2_len" value="${0.22 * scale}"/>
@@ -313,4 +313,54 @@
         <origin xyz="${ee_imu_x} ${ee_imu_y} ${ee_imu_z}" rpy="${ee_imu_roll} ${ee_imu_pitch} ${ee_imu_yaw}"/>
       </joint>
+      <gazebo reference="${prefix}ee_imu_link">
+        <sensor name="${prefix}ee_imu" type="imu">
+          <pose>0 0 0 0 0 0</pose>
+          <always_on>1</always_on>
+          <update_rate>100</update_rate>
+          <topic>${ee_imu_topic}</topic>
+          <imu>
+            <linear_acceleration>
+              <x>
+                <noise type="gaussian">
+                  <mean>0.0</mean>
+                  <stddev>0.01</stddev>
+                </noise>
+              </x>
+              <y>
+                <noise type="gaussian">
+                  <mean>0.0</mean>
+                  <stddev>0.01</stddev>
+                </noise>
+              </y>
+              <z>
+                <noise type="gaussian">
+                  <mean>0.0</mean>
+                  <stddev>0.01</stddev>
+                </noise>
+              </z>
+            </linear_acceleration>
+            <angular_velocity>
+              <x>
+                <noise type="gaussian">
+                  <mean>0.0</mean>
+                  <stddev>0.001</stddev>
+                </noise>
+              </x>
+              <y>
+                <noise type="gaussian">
+                  <mean>0.0</mean>
+                  <stddev>0.001</stddev>
+                </noise>
+              </y>
+              <z>
+                <noise type="gaussian">
+                  <mean>0.0</mean>
+                  <stddev>0.001</stddev>
+                </noise>
+              </z>
+            </angular_velocity>
+          </imu>
+        </sensor>
+      </gazebo>
     </xacro:if>
     <link name="${prefix}gripper_link">

File: clean_v2/ros2_ws/src/mm_robot_description/urdf/mm_robot.urdf.xacro (robot description, xacro)
@@ -136,4 +136,5 @@
     ee_imu_pitch="$(arg ee_imu_pitch)"
     ee_imu_yaw="$(arg ee_imu_yaw)"
+    ee_imu_topic="${ee_imu_topic}"
   />
   <joint name="${prefix}base_to_arm_joint" type="fixed">
@@ -231,57 +232,4 @@
         <update_rate>100</update_rate>
         <topic>$(eval '/' + namespace + '/imu_raw' if namespace != '' else '/imu_raw')</topic>
-        <imu>
-          <linear_acceleration>
-            <x>
-              <noise type="gaussian">
-                <mean>0.0</mean>
-                <stddev>0.01</stddev>
-              </noise>
-            </x>
-            <y>
-              <noise type="gaussian">
-                <mean>0.0</mean>
-                <stddev>0.01</stddev>
-              </noise>
-            </y>
-            <z>
-              <noise type="gaussian">
-                <mean>0.0</mean>
-                <stddev>0.01</stddev>
-              </noise>
-            </z>
-          </linear_acceleration>
-          <angular_velocity>
-            <x>
-              <noise type="gaussian">
-                <mean>0.0</mean>
-                <stddev>0.001</stddev>
-              </noise>
-            </x>
-            <y>
-              <noise type="gaussian">
-                <mean>0.0</mean>
-                <stddev>0.001</stddev>
-              </noise>
-            </y>
-            <z>
-              <noise type="gaussian">
-                <mean>0.0</mean>
-                <stddev>0.001</stddev>
-              </noise>
-            </z>
-          </angular_velocity>
-        </imu>
-      </sensor>
-    </gazebo>
-  </xacro:if>
-  <!-- IMU Sensor on end-effector link -->
-  <xacro:if value="$(arg enable_ee_imu)">
-    <gazebo reference="${prefix}ee_imu_link">
-      <sensor name="${prefix}ee_imu" type="imu">
-        <pose>0 0 0 0 0 0</pose>
-        <always_on>1</always_on>
-        <update_rate>100</update_rate>
-        <topic>${ee_imu_topic}</topic>
         <imu>
           <linear_acceleration>
