Commit message: fix: corregir topics de camaras en xacro
Evita error de xacro al calcular los topics y asegura rutas namespaced.

File: clean_v2/ros2_ws/src/mm_robot_description/urdf/mm_robot.urdf.xacro (robot description, xacro)
@@ -59,10 +59,9 @@
   <xacro:property name="controllers_file" value="$(arg controllers_file)"/>
   <xacro:property name="lidar_topic" value="$(eval '/' + namespace + '/scan' if namespace != '' else '/scan')"/>
-  <xacro:property name="camera_topic_prefix" value="$(eval '/' + namespace + '/camera' if namespace != '' else '/camera')"/>
-  <xacro:property name="cam_front_topic" value="$(eval camera_topic_prefix + '/front/image')"/>
-  <xacro:property name="cam_left_topic" value="$(eval camera_topic_prefix + '/left/image')"/>
-  <xacro:property name="cam_right_topic" value="$(eval camera_topic_prefix + '/right/image')"/>
-  <xacro:property name="cam_rear_topic" value="$(eval camera_topic_prefix + '/rear/image')"/>
-  <xacro:property name="ee_cam_topic" value="$(eval camera_topic_prefix + '/ee/image')"/>
+  <xacro:property name="cam_front_topic" value="$(eval '/' + namespace + '/camera/front/image' if namespace != '' else '/camera/front/image')"/>
+  <xacro:property name="cam_left_topic" value="$(eval '/' + namespace + '/camera/left/image' if namespace != '' else '/camera/left/image')"/>
+  <xacro:property name="cam_right_topic" value="$(eval '/' + namespace + '/camera/right/image' if namespace != '' else '/camera/right/image')"/>
+  <xacro:property name="cam_rear_topic" value="$(eval '/' + namespace + '/camera/rear/image' if namespace != '' else '/camera/rear/image')"/>
+  <xacro:property name="ee_cam_topic" value="$(eval '/' + namespace + '/camera/ee/image' if namespace != '' else '/camera/ee/image')"/>
   <xacro:mm_base
     prefix="${prefix}"

Commit message: fix: publicar camaras en image_raw
Alinea topicos de Gazebo con el bridge RAW para republish con frame_id correcto.

File: clean_v2/ros2_ws/src/mm_robot_description/urdf/mm_robot.urdf.xacro (robot description, xacro)
@@ -59,9 +59,9 @@
   <xacro:property name="controllers_file" value="$(arg controllers_file)"/>
   <xacro:property name="lidar_topic" value="$(eval '/' + namespace + '/scan' if namespace != '' else '/scan')"/>
-  <xacro:property name="cam_front_topic" value="$(eval '/' + namespace + '/camera/front/image' if namespace != '' else '/camera/front/image')"/>
-  <xacro:property name="cam_left_topic" value="$(eval '/' + namespace + '/camera/left/image' if namespace != '' else '/camera/left/image')"/>
-  <xacro:property name="cam_right_topic" value="$(eval '/' + namespace + '/camera/right/image' if namespace != '' else '/camera/right/image')"/>
-  <xacro:property name="cam_rear_topic" value="$(eval '/' + namespace + '/camera/rear/image' if namespace != '' else '/camera/rear/image')"/>
-  <xacro:property name="ee_cam_topic" value="$(eval '/' + namespace + '/camera/ee/image' if namespace != '' else '/camera/ee/image')"/>
+  <xacro:property name="cam_front_topic" value="$(eval '/' + namespace + '/camera/front/image_raw' if namespace != '' else '/camera/front/image_raw')"/>
+  <xacro:property name="cam_left_topic" value="$(eval '/' + namespace + '/camera/left/image_raw' if namespace != '' else '/camera/left/image_raw')"/>
+  <xacro:property name="cam_right_topic" value="$(eval '/' + namespace + '/camera/right/image_raw' if namespace != '' else '/camera/right/image_raw')"/>
+  <xacro:property name="cam_rear_topic" value="$(eval '/' + namespace + '/camera/rear/image_raw' if namespace != '' else '/camera/rear/image_raw')"/>
+  <xacro:property name="ee_cam_topic" value="$(eval '/' + namespace + '/camera/ee/image_raw' if namespace != '' else '/camera/ee/image_raw')"/>
   <xacro:mm_base
     prefix="${prefix}"

Commit message: Limpieza y correcciones MoveIt/IMU

File: clean_v2/ros2_ws/src/mm_robot_description/urdf/mm_robot.urdf.xacro (robot description, xacro)
@@ -56,4 +56,8 @@
   <xacro:arg name="ee_cam_pitch" default="0.0"/>
   <xacro:arg name="ee_cam_yaw" default="0.0"/>
+  <xacro:arg name="enable_imu" default="true"/>
+  <xacro:arg name="imu_x" default="0.0"/>
+  <xacro:arg name="imu_y" default="0.0"/>
+  <xacro:arg name="imu_z" default="0.10"/>
   <xacro:property name="prefix" value="$(arg prefix)"/>
   <xacro:property name="namespace" value="$(arg namespace)"/>
@@ -177,4 +181,83 @@
     </gazebo>
   </xacro:if>
+  <!-- IMU Sensor on base link -->
+  <xacro:if value="$(arg enable_imu)">
+    <link name="${prefix}imu_link">
+      <inertial>
+        <origin xyz="0 0 0" rpy="0 0 0"/>
+        <mass value="0.1"/>
+        <inertia ixx="0.0001" ixy="0" ixz="0" iyy="0.0001" iyz="0" izz="0.0001"/>
+      </inertial>
+      <xacro:if value="${base_visual_enabled}">
+        <visual>
+          <geometry>
+            <box size="0.05 0.05 0.05"/>
+          </geometry>
+          <material name="SensorBlack">
+            <color rgba="0.1 0.1 0.1 1.0"/>
+          </material>
+        </visual>
+      </xacro:if>
+      <collision>
+        <geometry>
+          <box size="0.05 0.05 0.05"/>
+        </geometry>
+      </collision>
+    </link>
+    <joint name="${prefix}imu_joint" type="fixed">
+      <parent link="${prefix}base_link"/>
+      <child link="${prefix}imu_link"/>
+      <origin xyz="$(arg imu_x) $(arg imu_y) $(arg imu_z)" rpy="0 0 0"/>
+    </joint>
+    <gazebo reference="${prefix}imu_link">
+      <sensor name="${prefix}imu" type="imu">
+        <pose>0 0 0 0 0 0</pose>
+        <update_rate>100</update_rate>
+        <topic>$(eval '/' + namespace + '/imu' if namespace != '' else '/imu')</topic>
+        <imu>
+          <linear_acceleration>
+            <x>
+              <noise type="gaussian">
+                <mean>0.0</mean>
+                <stddev>0.01</stddev>
+              </noise>
+            </x>
+            <y>
+              <noise type="gaussian">
+                <mean>0.0</mean>
+                <stddev>0.01</stddev>
+              </noise>
+            </y>
+            <z>
+              <noise type="gaussian">
+                <mean>0.0</mean>
+                <stddev>0.01</stddev>
+              </noise>
+            </z>
+          </linear_acceleration>
+          <angular_velocity>
+            <x>
+              <noise type="gaussian">
+                <mean>0.0</mean>
+                <stddev>0.001</stddev>
+              </noise>
+            </x>
+            <y>
+              <noise type="gaussian">
+                <mean>0.0</mean>
+                <stddev>0.001</stddev>
+              </noise>
+            </y>
+            <z>
+              <noise type="gaussian">
+                <mean>0.0</mean>
+                <stddev>0.001</stddev>
+              </noise>
+            </z>
+          </angular_velocity>
+        </imu>
+      </sensor>
+    </gazebo>
+  </xacro:if>
   <gazebo reference="${prefix}cam_front_link">
     <sensor name="${prefix}cam_front" type="camera">

Commit message: fix(bringup): lidar republisher y ajustes ekf/rviz/imu

File: clean_v2/ros2_ws/src/mm_robot_description/urdf/mm_robot.urdf.xacro (robot description, xacro)
@@ -60,5 +60,5 @@
   <xacro:arg name="imu_y" default="0.0"/>
   <xacro:arg name="imu_z" default="0.10"/>
-  <xacro:arg name="enable_ee_imu" default="true"/>
+  <xacro:arg name="enable_ee_imu" default="false"/>
   <xacro:arg name="ee_imu_x" default="0.03"/>
   <xacro:arg name="ee_imu_y" default="0.0"/>
@@ -76,5 +76,5 @@
   <xacro:property name="arm_mount_z" value="${(base_height / 2.0) + arm_mount_height}"/>
   <xacro:property name="base_visual_enabled" value="${visual_mode == 'full' or visual_mode == 'base_only'}"/>
-  <xacro:property name="lidar_topic" value="$(eval '/' + namespace + '/scan' if namespace != '' else '/scan')"/>
+  <xacro:property name="lidar_topic" value="$(eval '/' + namespace + '/scan_raw' if namespace != '' else '/scan_raw')"/>
   <xacro:property name="cam_front_topic" value="$(eval '/' + namespace + '/camera/front/image_raw' if namespace != '' else '/camera/front/image_raw')"/>
   <xacro:property name="cam_left_topic" value="$(eval '/' + namespace + '/camera/left/image_raw' if namespace != '' else '/camera/left/image_raw')"/>

Commit message: feat(sim): add EE IMU link opt-in and clarify health warnings

File: clean_v2/ros2_ws/src/mm_robot_description/urdf/mm_robot.urdf.xacro (robot description, xacro)
@@ -278,4 +278,16 @@
   <!-- IMU Sensor on end-effector link -->
   <xacro:if value="$(arg enable_ee_imu)">
+    <link name="${prefix}ee_imu_link">
+      <inertial>
+        <origin xyz="0 0 0" rpy="0 0 0"/>
+        <mass value="0.05"/>
+        <inertia ixx="0.00005" ixy="0" ixz="0" iyy="0.00005" iyz="0" izz="0.00005"/>
+      </inertial>
+    </link>
+    <joint name="${prefix}ee_imu_joint" type="fixed">
+      <parent link="${prefix}tool0"/>
+      <child link="${prefix}ee_imu_link"/>
+      <origin xyz="$(arg ee_imu_x) $(arg ee_imu_y) $(arg ee_imu_z)" rpy="$(arg ee_imu_roll) $(arg ee_imu_pitch) $(arg ee_imu_yaw)"/>
+    </joint>
     <gazebo reference="${prefix}ee_imu_link">
       <sensor name="${prefix}ee_imu" type="imu">

Commit message: feat(sim): enable ee imu and avoid duplicate ee_imu_link

File: clean_v2/ros2_ws/src/mm_robot_description/urdf/mm_robot.urdf.xacro (robot description, xacro)
@@ -278,16 +278,4 @@
   <!-- IMU Sensor on end-effector link -->
   <xacro:if value="$(arg enable_ee_imu)">
-    <link name="${prefix}ee_imu_link">
-      <inertial>
-        <origin xyz="0 0 0" rpy="0 0 0"/>
-        <mass value="0.05"/>
-        <inertia ixx="0.00005" ixy="0" ixz="0" iyy="0.00005" iyz="0" izz="0.00005"/>
-      </inertial>
-    </link>
-    <joint name="${prefix}ee_imu_joint" type="fixed">
-      <parent link="${prefix}tool0"/>
-      <child link="${prefix}ee_imu_link"/>
-      <origin xyz="$(arg ee_imu_x) $(arg ee_imu_y) $(arg ee_imu_z)" rpy="$(arg ee_imu_roll) $(arg ee_imu_pitch) $(arg ee_imu_yaw)"/>
-    </joint>
     <gazebo reference="${prefix}ee_imu_link">
       <sensor name="${prefix}ee_imu" type="imu">
